Commit message: Images for choosing the height and angle of camera

File: robot_description/urdf/robot_final.gazebo.macro.xacro (robot description, xacro)
@@ -166,6 +166,6 @@
 <!--              <width>640</width>-->
 <!--              <height>480</height>-->
-             <width>1680</width>
-              <height>1050</height>
+             <width>680</width>
+              <height>480</height>
               <format>R8G8B8</format>
           </image>

File: robot_description/urdf/robot_final.urdf.xacro (robot description, xacro)
@@ -242,5 +242,5 @@
   </link>
   <joint name="camera_rgb_joint" type="fixed">
-    <origin xyz="0.003 0.011 0.009" rpy="0 0 0"/>
+    <origin xyz="0.003 0.011 0.6" rpy="0 0.6 0"/>
     <parent link="camera_link"/>
     <child link="camera_rgb_frame"/>

Commit message: new_models and new robot (on progress) for gazebo

File: robot_description/urdf/robot_final.gazebo.macro.xacro (robot description, xacro)
@@ -1,4 +1,5 @@
 <?xml version="1.0"?>
 <robot name="robot_gaz" xmlns:xacro="http://ros.org/wiki/xacro">
+  <!-- <xacro:include filename="$(find robot_description)/urdf/Skid_steering_drive.xacro"/> -->
   <xacro:include filename="$(find robot_description)/urdf/ros_diff_drive.gazebo.xacro"/>
 <!--  <xacro:include filename="$(find p_g5_description)/urdf/ros_control.gazebo.xacro"/>-->
@@ -13,5 +14,5 @@
     <mu2>0.1</mu2>
     <kp>500000.0</kp>
-    <kd>10.0</kd>
+    <kd>10000.0</kd>
     <minDepth>0.001</minDepth>
     <maxVel>0.1</maxVel>
@@ -20,18 +21,18 @@
   </gazebo>
   <gazebo reference="wheel_left_front_link">
+    <mu1>0</mu1>
+    <mu2>0</mu2>
+    <!-- <kp>500000.0</kp>
+    <kd>10000.0</kd>
+    <minDepth>0.001</minDepth>
+    <maxVel>0.1</maxVel>
+    <fdir1>1 0 0</fdir1> -->
+    <material>Gazebo/${player_color}</material>
+  </gazebo>
+  <gazebo reference="wheel_right_link">
     <mu1>0.1</mu1>
     <mu2>0.1</mu2>
     <kp>500000.0</kp>
-    <!-- <kd>10.0</kd>
-    <minDepth>0.001</minDepth>
-    <maxVel>0.1</maxVel>
-    <fdir1>1 0 0</fdir1> -->
-    <material>Gazebo/${player_color}</material>
-  </gazebo>
-  <gazebo reference="wheel_right_link">
-    <mu1>0.1</mu1>
-    <mu2>0.1</mu2>
-    <kp>500000.0</kp>
-    <kd>10.0</kd>
+    <kd>10000.0</kd>
     <minDepth>0.001</minDepth>
     <maxVel>0.1</maxVel>
@@ -40,8 +41,8 @@
   </gazebo>
   <gazebo reference="wheel_right_front_link">
-    <mu1>0.1</mu1>
-    <mu2>0.1</mu2>
-    <kp>500000.0</kp>
-    <!-- <kd>10.0</kd>
+    <mu1>0</mu1>
+    <mu2>0</mu2>
+    <!-- <kp>500000.0</kp>
+    <kd>10000.0</kd>
     <minDepth>0.001</minDepth>
     <maxVel>0.1</maxVel>

File: robot_description/urdf/robot_final.urdf.xacro (robot description, xacro)
@@ -17,22 +17,24 @@
     <parent link="base_footprint"/>
     <child link="base_link" />
-    <origin xyz="0 0 0.010" rpy="0 0 ${orientacao}"/>
+    <origin xyz="0 0 0.0624" rpy="0 0 0"/>
   </joint>
   <link name="base_link">
     <visual>
-      <origin xyz="-0.064 0 0.0" rpy="0 0 0"/>
-      <geometry>
-        <mesh filename="package://turtlebot3_description/meshes/bases/waffle_pi_base.stl" scale="0.001 0.001 0.001"/>
+      <!-- <origin xyz="-0.064 0 0.0" rpy="0 0 0"/> -->
+      <origin xyz="0 0 0" rpy="1.57 0 0"/>
+      <geometry>
+        <!-- <mesh filename="package://turtlebot3_description/meshes/bases/waffle_pi_base.stl" scale="0.001 0.001 0.001"/> -->
+        <mesh filename="$(find robot_description)/meshes/base_link.STL" scale="0.001 0.001 0.001"/>
       </geometry>
       <material name="${base_color}"/>
     </visual>
     <collision>
-      <origin xyz="-0.064 0 0.047" rpy="0 0 0"/>
-      <geometry>
-        <box size="0.266 0.266 0.094"/>
-      </geometry>
-    </collision>
-    <inertial>
-      <origin xyz="0 0 0" rpy="0 0 0"/>
+      <origin xyz="0.162 -0.125 0.020" rpy="0 0 0"/>
+      <geometry>
+        <box size="0.32 0.16 0.040"/>
+      </geometry>
+    </collision>
+    <inertial>
+      <origin xyz="0.162 -0.1315 0.020" rpy="0 0 0"/>
       <mass value="1.3729096e+00"/>
       <inertia ixx="8.7002718e-03" ixy="-4.7576583e-05" ixz="1.1160499e-04"
@@ -44,25 +46,23 @@
     <parent link="base_link"/>
     <child link="wheel_left_link"/>
-    <origin xyz="0.0 0.144 0.023" rpy="-1.57 0 0"/>
-    <axis xyz="0 0 1"/>
+    <origin xyz="0.0124 0.0 0.0123" rpy="0 0 0"/>
+    <axis xyz="0 1 0"/>
   </joint>
   <link name="wheel_left_link">
     <visual>
-      <origin xyz="0 0 0" rpy="1.57 0 0"/>
-      <!-- <origin xyz="0 0 0" rpy="1.57 1.57 0"/> -->
-      <geometry>
-        <mesh filename="package://turtlebot3_description/meshes/wheels/left_tire.stl" scale="0.001 0.001 0.001"/>
-        <!-- <mesh filename="$(find robot_description)/meshes/Disk_5.stl" scale="0.0004 0.0004 0.0004"/> -->
-      </geometry>
-      <material name="${player_color}"/>
-    </visual>
-    <collision>
-      <origin xyz="0 0 0" rpy="0 0 0"/>
-      <geometry>
-        <cylinder length="0.018" radius="0.033"/>
-      </geometry>
-    </collision>
-    <inertial>
-      <origin xyz="0 0 0" />
+      <origin xyz="-0.0624 0 -0.0624" rpy="1.57 0 0"/>
+      <geometry>
+        <mesh filename="$(find robot_description)/meshes/Wheel.STL" scale="0.001 0.001 0.001"/>
+      </geometry>
+      <material name="${player_color}"/>
+    </visual>
+    <collision>
+      <origin xyz="0 -0.0215 0" rpy="1.57 0 0"/>
+      <geometry>
+        <cylinder length="0.045" radius="0.0624"/>
+      </geometry>
+    </collision>
+    <inertial>
+      <origin xyz="0.0 -0.0225 0.0124 " />
       <mass value="2.8498940e-02" />
       <inertia ixx="1.1175580e-05" ixy="-4.2369783e-11" ixz="-5.9381719e-09"
@@ -71,28 +71,27 @@
       </inertial>
   </link>
+<!-- wheel_left_front_joint -->
   <joint name="wheel_left_front_joint" type="continuous">
     <parent link="base_link"/>
     <child link="wheel_left_front_link"/>
-    <origin xyz="-0.135 0.144 0.023" rpy="-1.57 0 0"/>
-    <axis xyz="0 0 1"/>
+    <origin xyz="0.3124 0.0 0.0123" rpy="0 0 0"/>
+    <axis xyz="0 1 0"/>
   </joint>
   <link name="wheel_left_front_link">
     <visual>
-      <!-- <origin xyz="0 0 0" rpy="1.57 1.57 0"/> -->
-      <origin xyz="0 0 0" rpy="1.57 1.57 0"/>
-      <geometry>
-        <!-- <mesh filename="package://turtlebot3_description/meshes/wheels/left_tire.stl" scale="0.001 0.001 0.001"/> -->
-        <mesh filename="$(find robot_description)/meshes/Disk_5.stl" scale="0.0004 0.0004 0.0004"/>
-      </geometry>
-      <material name="${player_color}"/>
-    </visual>
-    <collision>
-      <origin xyz="0 0 0" rpy="0 0 0"/>
-      <geometry>
-        <cylinder length="0.018" radius="0.033"/>
-      </geometry>
-    </collision>
-    <inertial>
-      <origin xyz="0 0 0" />
+      <origin xyz="-0.0624 0 -0.0624" rpy="1.57 0 0"/>
+      <geometry>
+        <mesh filename="$(find robot_description)/meshes/Wheel.STL" scale="0.001 0.001 0.001"/>
+      </geometry>
+      <material name="${player_color}"/>
+    </visual>
+    <collision>
+      <origin xyz="0 -0.0215 0" rpy="1.57 0 0"/>
+      <geometry>
+        <cylinder length="0.045" radius="0.0624"/>
+      </geometry>
+    </collision>
+    <inertial>
+      <origin xyz="0.0 -0.0225 0.0124 " />
       <mass value="2.8498940e-02" />
       <inertia ixx="1.1175580e-05" ixy="-4.2369783e-11" ixz="-5.9381719e-09"
@@ -101,29 +100,27 @@
       </inertial>
   </link>
+  <!-- wheel_right_joint -->
   <joint name="wheel_right_joint" type="continuous">
     <parent link="base_link"/>
     <child link="wheel_right_link"/>
-    <origin xyz="0.0 -0.144 0.023" rpy="-1.57 0 0"/>
-    <axis xyz="0 0 1"/>
+    <origin xyz="0.0124 -0.251 0.0123" rpy="0 0 0"/>
+    <axis xyz="0 1 0"/>
   </joint>
   <link name="wheel_right_link">
     <visual>
-      <origin xyz="0 0 0" rpy="1.57 0 0"/>
-      <!-- <origin xyz="0 0 0" rpy="1.57 1.57 0"/> -->
-      <geometry>
-        <mesh filename="package://turtlebot3_description/meshes/wheels/right_tire.stl" scale="0.001 0.001 0.001"/>
-        <!-- <mesh filename="$(find robot_description)/meshes/Disk_5.stl" scale="0.0004 0.0004 0.0004"/> -->
-      </geometry>
-<!--      <material name="dark"/>-->
-      <material name="${player_color}"/>
-    </visual>
-    <collision>
-      <origin xyz="0 0 0" rpy="0 0 0"/>
-      <geometry>
-        <cylinder length="0.018" radius="0.033"/>
-      </geometry>
-    </collision>
-    <inertial>
-      <origin xyz="0 0 0" />
+      <origin xyz="0.0624 0 -0.0624" rpy="1.57 0 3.14"/>
+      <geometry>
+        <mesh filename="$(find robot_description)/meshes/Wheel.STL" scale="0.001 0.001 0.001"/>
+      </geometry>
+      <material name="${player_color}"/>
+    </visual>
+    <collision>
+      <origin xyz="0 0.0215 0" rpy="1.57 0 0"/>
+      <geometry>
+        <cylinder length="0.045" radius="0.0624"/>
+      </geometry>
+    </collision>
+    <inertial>
+      <origin xyz="0.0 -0.0225 0.0124 " />
       <mass value="2.8498940e-02" />
       <inertia ixx="1.1175580e-05" ixy="-4.2369783e-11" ixz="-5.9381719e-09"
@@ -132,35 +129,34 @@
       </inertial>
   </link>
-  <joint name="wheel_right_front_joint" type="continuous">
-    <parent link="base_link"/>
-    <child link="wheel_right_front_link"/>
-    <origin xyz="-0.135 -0.144 0.023" rpy="-1.57 0 0"/>
-    <axis xyz="0 0 1"/>
-  </joint>
-  <link name="wheel_right_front_link">
-    <visual>
-      <!-- <origin xyz="0 0 0" rpy="1.57 0 0"/> -->
-      <origin xyz="0 0 0" rpy="1.57 1.57 0"/>
-      <geometry>
-        <!-- <mesh filename="package://turtlebot3_description/meshes/wheels/right_tire.stl" scale="0.001 0.001 0.001"/> -->
-        <mesh filename="$(find robot_description)/meshes/Disk_5.stl" scale="0.0004 0.0004 0.0004"/>
-      </geometry>
-<!--      <material name="dark"/>-->
-      <material name="${player_color}"/>
-    </visual>
-    <collision>
-      <origin xyz="0 0 0" rpy="0 0 0"/>
-      <geometry>
-        <cylinder length="0.018" radius="0.033"/>
-      </geometry>
-    </collision>
-    <inertial>
-      <origin xyz="0 0 0" />
-      <mass value="2.8498940e-02" />
-      <inertia ixx="1.1175580e-05" ixy="-4.2369783e-11" ixz="-5.9381719e-09"
-               iyy="1.1192413e-05" iyz="-1.4400107e-11"
-               izz="2.0712558e-05" />
-      </inertial>
-  </link>
+  <!-- wheel_right_front_joint -->
+ <joint name="wheel_right_front_joint" type="continuous">
+  <parent link="base_link"/>
+  <child link="wheel_right_front_link"/>
+  <origin xyz="0.3124 -0.251 0.0123" rpy="0 0 0"/>
+  <axis xyz="0 1 0"/>
+</joint>
+<link name="wheel_right_front_link">
+  <visual>
+    <origin xyz="0.0624 0 -0.0624" rpy="1.57 0 3.14"/>
+    <geometry>
+      <mesh filename="$(find robot_description)/meshes/Wheel.STL" scale="0.001 0.001 0.001"/>
+    </geometry>
+    <material name="${player_color}"/>
+  </visual>
+  <collision>
+    <origin xyz="0 0.0215 0" rpy="1.57 0 0"/>
+    <geometry>
+      <cylinder length="0.045" radius="0.0624"/>
+    </geometry>
+  </collision>
+  <inertial>
+    <origin xyz="0.0 -0.0225 0.0124 " />
+    <mass value="2.8498940e-02" />
+    <inertia ixx="1.1175580e-05" ixy="-4.2369783e-11" ixz="-5.9381719e-09"
+             iyy="1.1192413e-05" iyz="-1.4400107e-11"
+             izz="2.0712558e-05" />
+    </inertial>
+</link>
+<!--
   <joint name="caster_back_right_joint" type="fixed">
     <parent link="base_link"/>
@@ -183,4 +179,6 @@
     </inertial>
   </link>
+ -->
+<!--
   <joint name="caster_back_left_joint" type="fixed">
     <parent link="base_link"/>
@@ -203,4 +201,6 @@
     </inertial>
   </link>
+ -->
+<!--
   <joint name="imu_joint" type="fixed">
     <parent link="base_link"/>
@@ -209,4 +209,6 @@
   </joint>
   <link name="imu_link"/>
+-->
+<!--
   <joint name="scan_joint" type="fixed">
     <parent link="base_link"/>
@@ -236,4 +238,6 @@
     </inertial>
   </link>
+-->
+<!--
   <joint name="camera_joint" type="fixed">
     <origin xyz="0.073 -0.011 0.084" rpy="0 0 0"/>
@@ -249,10 +253,14 @@
     </collision>
   </link>
+-->
+<!--
   <joint name="camera_rgb_joint" type="fixed">
-    <origin xyz="0.003 0.011 0.6" rpy="0 0.6 0"/>    -  <!-- old values <origin xyz="0.003 0.011 0.45" rpy="0 0.15 0"/> --> <!-- <origin xyz="0.003 0.011 0.45" rpy="0 0.38 0"/>-->
+    <origin xyz="0.003 0.011 0.6" rpy="0 0.6 0"/>
     <parent link="camera_link"/>
     <child link="camera_rgb_frame"/>
   </joint>
   <link name="camera_rgb_frame"/>
+ -->
+<!--
   <joint name="camera_rgb_optical_joint" type="fixed">
     <origin xyz="0 0 0" rpy="-1.57 0 -1.57"/>
@@ -261,3 +269,4 @@
   </joint>
   <link name="camera_rgb_optical_frame"/>
+-->
 </robot>

Commit message: Robot Final

File: robot_description/urdf/robot_final.gazebo.macro.xacro (robot description, xacro)
@@ -159,4 +159,5 @@
 <!--link : https://www.raspberrypi.org/documentation/hardware/camera/-->
   <gazebo reference="camera_rgb_frame">
+    <material>Gazebo/${base_color}</material>
     <sensor type="camera" name="Pi Camera">
       <always_on>true</always_on>

File: robot_description/urdf/robot_final.urdf.xacro (robot description, xacro)
@@ -210,22 +210,22 @@
   <link name="imu_link"/>
 -->
-<!--
+<!-- Scan base sensors -->
   <joint name="scan_joint" type="fixed">
     <parent link="base_link"/>
     <child link="base_scan"/>
-    <origin xyz="-0.064 0 0.122" rpy="0 0 0"/>
+    <origin xyz="0 0 0.0624" rpy="0 0 0"/>
   </joint>
   <link name="base_scan">
     <visual>
-      <origin xyz="0 0 0.0" rpy="0 0 0"/>
-      <geometry>
-        <mesh filename="package://turtlebot3_description/meshes/sensors/lds.stl" scale="0.001 0.001 0.001"/>
-      </geometry>
-      <material name="${player_color}"/>
-    </visual>
-    <collision>
-      <origin xyz="0.015 0 -0.0065" rpy="0 0 0"/>
-      <geometry>
-        <cylinder length="0.0315" radius="0.055"/>
+      <origin xyz="-0.136 0.0289 -0.025" rpy="1.57 0 0"/>
+      <geometry>
+        <mesh filename="$(find robot_description)/meshes/base_scan_sensors.STL" scale="0.001 0.001 0.001"/>
+      </geometry>
+      <material name="${player_color}"/>
+    </visual>
+    <collision>
+      <origin xyz="0.15 -0.15 0.25" rpy="0 0 0"/>
+      <geometry>
+        <box size="0.6 0.350 0.425"/>
       </geometry>
     </collision>
@@ -238,6 +238,5 @@
     </inertial>
   </link>
--->
-<!--
+  <!-- Camera link -->
   <joint name="camera_joint" type="fixed">
     <origin xyz="0.073 -0.011 0.084" rpy="0 0 0"/>
@@ -246,27 +245,33 @@
   </joint>
   <link name="camera_link">
-    <collision>
-      <origin xyz="0.005 0.011 0.013" rpy="0 0 0"/>
-      <geometry>
-        <box size="0.015 0.030 0.027"/>
-      </geometry>
-    </collision>
-  </link>
--->
-<!--
+  </link>
+  <!-- camera_rgb_joint -->
   <joint name="camera_rgb_joint" type="fixed">
-    <origin xyz="0.003 0.011 0.6" rpy="0 0.6 0"/>
+    <!-- <origin xyz="0.003 0.011 0.6" rpy="0 0.6 0"/>     -->
+    <origin xyz="0.3 0.011 0.45" rpy="0 0.6 0"/>
     <parent link="camera_link"/>
     <child link="camera_rgb_frame"/>
   </joint>
-  <link name="camera_rgb_frame"/>
- -->
-<!--
-  <joint name="camera_rgb_optical_joint" type="fixed">
+  <link name="camera_rgb_frame">
+    <visual>
+      <origin xyz="0 0 0 " rpy="1.6 0 0"/>
+      <geometry>
+        <mesh filename="$(find robot_description)/meshes/kinet.STL" scale="0.001 0.001 0.001"/>
+      </geometry>
+      <material name="${base_color}"/>
+    </visual>
+    <collision>
+      <origin xyz="0 0 0" rpy="0 0 0"/>
+      <geometry>
+        <box size="0.1 0.3 0.1"/>
+      </geometry>
+    </collision>
+      </link>
+  <!-- camera_rgb_optical_joint -->
+  <!-- <joint name="camera_rgb_optical_joint" type="fixed">
     <origin xyz="0 0 0" rpy="-1.57 0 -1.57"/>
     <parent link="camera_rgb_frame"/>
     <child link="camera_rgb_optical_frame"/>
   </joint>
-  <link name="camera_rgb_optical_frame"/>
--->
+  <link name="camera_rgb_optical_frame"/>  -->
 </robot>
