Commit message: meshes for robot

File: robot_description/urdf/robot_final.urdf.xacro (robot description, xacro)
@@ -49,7 +49,9 @@
   <link name="wheel_left_link">
     <visual>
-      <origin xyz="0 0 0" rpy="1.57 0 0"/>
-      <geometry>
-        <mesh filename="package://turtlebot3_description/meshes/wheels/left_tire.stl" scale="0.001 0.001 0.001"/>
+      <!-- <origin xyz="0 0 0" rpy="1.57 0 0"/> -->
+      <origin xyz="0 0 0" rpy="1.57 1.57 0"/>
+      <geometry>
+        <!-- <mesh filename="package://turtlebot3_description/meshes/wheels/left_tire.stl" scale="0.001 0.001 0.001"/> -->
+        <mesh filename="$(find robot_description)/meshes/Disk_5.stl" scale="0.0004 0.0004 0.0004"/>
       </geometry>
       <material name="${player_color}"/>
@@ -77,7 +79,9 @@
   <link name="wheel_left_front_link">
     <visual>
-      <origin xyz="0 0 0" rpy="1.57 0 0"/>
-      <geometry>
-        <mesh filename="package://turtlebot3_description/meshes/wheels/left_tire.stl" scale="0.001 0.001 0.001"/>
+      <!-- <origin xyz="0 0 0" rpy="1.57 1.57 0"/> -->
+      <origin xyz="0 0 0" rpy="1.57 1.57 0"/>
+      <geometry>
+        <!-- <mesh filename="package://turtlebot3_description/meshes/wheels/left_tire.stl" scale="0.001 0.001 0.001"/> -->
+        <mesh filename="$(find robot_description)/meshes/Disk_5.stl" scale="0.0004 0.0004 0.0004"/>
       </geometry>
       <material name="${player_color}"/>
@@ -105,7 +109,9 @@
   <link name="wheel_right_link">
     <visual>
-      <origin xyz="0 0 0" rpy="1.57 0 0"/>
-      <geometry>
-        <mesh filename="package://turtlebot3_description/meshes/wheels/right_tire.stl" scale="0.001 0.001 0.001"/>
+      <!-- <origin xyz="0 0 0" rpy="1.57 0 0"/> -->
+      <origin xyz="0 0 0" rpy="1.57 1.57 0"/>
+      <geometry>
+        <!-- <mesh filename="package://turtlebot3_description/meshes/wheels/right_tire.stl" scale="0.001 0.001 0.001"/> -->
+        <mesh filename="$(find robot_description)/meshes/Disk_5.stl" scale="0.0004 0.0004 0.0004"/>
       </geometry>
 <!--      <material name="dark"/>-->
@@ -134,7 +140,9 @@
   <link name="wheel_right_front_link">
     <visual>
-      <origin xyz="0 0 0" rpy="1.57 0 0"/>
-      <geometry>
-        <mesh filename="package://turtlebot3_description/meshes/wheels/right_tire.stl" scale="0.001 0.001 0.001"/>
+      <!-- <origin xyz="0 0 0" rpy="1.57 0 0"/> -->
+      <origin xyz="0 0 0" rpy="1.57 1.57 0"/>
+      <geometry>
+        <!-- <mesh filename="package://turtlebot3_description/meshes/wheels/right_tire.stl" scale="0.001 0.001 0.001"/> -->
+        <mesh filename="$(find robot_description)/meshes/Disk_5.stl" scale="0.0004 0.0004 0.0004"/>
       </geometry>
 <!--      <material name="dark"/>-->

Commit message: Vision Program advancement- Aplicação do código para reconehcer linhas a aprtir de uma área de interesse triangular; -Receção e tratamento da imagem da câmara do robot.

File: robot_description/urdf/robot_final.urdf.xacro (robot description, xacro)
@@ -250,5 +250,5 @@
   </link>
   <joint name="camera_rgb_joint" type="fixed">
-    <origin xyz="0.003 0.011 0.6" rpy="0 0.6 0"/>
+   <origin xyz="0.003 0.011 0.6" rpy="0 0 0"/>       <!-- old values (SF):xyz="0.003 0.011 0.6" rpy="0 0.6 0"-->
     <parent link="camera_link"/>
     <child link="camera_rgb_frame"/>

Commit message: urdf ready for update

File: robot_description/urdf/robot_final.urdf.xacro (robot description, xacro)
@@ -49,5 +49,35 @@
   <link name="wheel_left_link">
     <visual>
-      <!-- <origin xyz="0 0 0" rpy="1.57 0 0"/> -->
+      <origin xyz="0 0 0" rpy="1.57 0 0"/>
+      <!-- <origin xyz="0 0 0" rpy="1.57 1.57 0"/> -->
+      <geometry>
+        <mesh filename="package://turtlebot3_description/meshes/wheels/left_tire.stl" scale="0.001 0.001 0.001"/>
+        <!-- <mesh filename="$(find robot_description)/meshes/Disk_5.stl" scale="0.0004 0.0004 0.0004"/> -->
+      </geometry>
+      <material name="${player_color}"/>
+    </visual>
+    <collision>
+      <origin xyz="0 0 0" rpy="0 0 0"/>
+      <geometry>
+        <cylinder length="0.018" radius="0.033"/>
+      </geometry>
+    </collision>
+    <inertial>
+      <origin xyz="0 0 0" />
+      <mass value="2.8498940e-02" />
+      <inertia ixx="1.1175580e-05" ixy="-4.2369783e-11" ixz="-5.9381719e-09"
+               iyy="1.1192413e-05" iyz="-1.4400107e-11"
+               izz="2.0712558e-05" />
+      </inertial>
+  </link>
+  <joint name="wheel_left_front_joint" type="continuous">
+    <parent link="base_link"/>
+    <child link="wheel_left_front_link"/>
+    <origin xyz="-0.135 0.144 0.023" rpy="-1.57 0 0"/>
+    <axis xyz="0 0 1"/>
+  </joint>
+  <link name="wheel_left_front_link">
+    <visual>
+      <!-- <origin xyz="0 0 0" rpy="1.57 1.57 0"/> -->
       <origin xyz="0 0 0" rpy="1.57 1.57 0"/>
       <geometry>
@@ -71,34 +101,4 @@
       </inertial>
   </link>
-  <joint name="wheel_left_front_joint" type="continuous">
-    <parent link="base_link"/>
-    <child link="wheel_left_front_link"/>
-    <origin xyz="-0.135 0.144 0.023" rpy="-1.57 0 0"/>
-    <axis xyz="0 0 1"/>
-  </joint>
-  <link name="wheel_left_front_link">
-    <visual>
-      <!-- <origin xyz="0 0 0" rpy="1.57 1.57 0"/> -->
-      <origin xyz="0 0 0" rpy="1.57 1.57 0"/>
-      <geometry>
-        <!-- <mesh filename="package://turtlebot3_description/meshes/wheels/left_tire.stl" scale="0.001 0.001 0.001"/> -->
-        <mesh filename="$(find robot_description)/meshes/Disk_5.stl" scale="0.0004 0.0004 0.0004"/>
-      </geometry>
-      <material name="${player_color}"/>
-    </visual>
-    <collision>
-      <origin xyz="0 0 0" rpy="0 0 0"/>
-      <geometry>
-        <cylinder length="0.018" radius="0.033"/>
-      </geometry>
-    </collision>
-    <inertial>
-      <origin xyz="0 0 0" />
-      <mass value="2.8498940e-02" />
-      <inertia ixx="1.1175580e-05" ixy="-4.2369783e-11" ixz="-5.9381719e-09"
-               iyy="1.1192413e-05" iyz="-1.4400107e-11"
-               izz="2.0712558e-05" />
-      </inertial>
-  </link>
   <joint name="wheel_right_joint" type="continuous">
     <parent link="base_link"/>
@@ -109,9 +109,9 @@
   <link name="wheel_right_link">
     <visual>
-      <!-- <origin xyz="0 0 0" rpy="1.57 0 0"/> -->
-      <origin xyz="0 0 0" rpy="1.57 1.57 0"/>
-      <geometry>
-        <!-- <mesh filename="package://turtlebot3_description/meshes/wheels/right_tire.stl" scale="0.001 0.001 0.001"/> -->
-        <mesh filename="$(find robot_description)/meshes/Disk_5.stl" scale="0.0004 0.0004 0.0004"/>
+      <origin xyz="0 0 0" rpy="1.57 0 0"/>
+      <!-- <origin xyz="0 0 0" rpy="1.57 1.57 0"/> -->
+      <geometry>
+        <mesh filename="package://turtlebot3_description/meshes/wheels/right_tire.stl" scale="0.001 0.001 0.001"/>
+        <!-- <mesh filename="$(find robot_description)/meshes/Disk_5.stl" scale="0.0004 0.0004 0.0004"/> -->
       </geometry>
 <!--      <material name="dark"/>-->

Commit message: Upload ML_approach

File: robot_description/urdf/robot_final.urdf.xacro (robot description, xacro)
@@ -250,5 +250,5 @@
   </link>
   <joint name="camera_rgb_joint" type="fixed">
-    <origin xyz="0.003 0.011 0.45" rpy="0 0.15 0"/>    -  <!-- old values (SF):xyz="0.003 0.011 0.6" rpy="0 0.6 0"-->
+    <origin xyz="0.003 0.011 0.6" rpy="0 0.6 0"/>    -  <!-- old values <origin xyz="0.003 0.011 0.45" rpy="0 0.15 0"/> -->
     <parent link="camera_link"/>
     <child link="camera_rgb_frame"/>

Commit message: Tentativa polyfit

File: robot_description/urdf/robot_final.urdf.xacro (robot description, xacro)
@@ -250,5 +250,5 @@
   </link>
   <joint name="camera_rgb_joint" type="fixed">
-    <origin xyz="0.003 0.011 0.6" rpy="0 0.6 0"/>    -  <!-- old values <origin xyz="0.003 0.011 0.45" rpy="0 0.15 0"/> -->
+    <origin xyz="0.003 0.011 0.45" rpy="0 0.38 0"/>    -  <!-- old values <origin xyz="0.003 0.011 0.45" rpy="0 0.15 0"/> -->
     <parent link="camera_link"/>
     <child link="camera_rgb_frame"/>

Commit message: Change camera position

File: robot_description/urdf/robot_final.urdf.xacro (robot description, xacro)
@@ -250,5 +250,5 @@
   </link>
   <joint name="camera_rgb_joint" type="fixed">
-    <origin xyz="0.003 0.011 0.45" rpy="0 0.38 0"/>    -  <!-- old values <origin xyz="0.003 0.011 0.45" rpy="0 0.15 0"/> -->
+    <origin xyz="0.003 0.011 0.6" rpy="0 0.6 0"/>    -  <!-- old values <origin xyz="0.003 0.011 0.45" rpy="0 0.15 0"/> --> <!-- <origin xyz="0.003 0.011 0.45" rpy="0 0.38 0"/>-->
     <parent link="camera_link"/>
     <child link="camera_rgb_frame"/>

Commit message: New training file

File: robot_description/urdf/robot_final.urdf.xacro (robot description, xacro)
@@ -210,4 +210,12 @@
   <link name="imu_link"/>
 -->
+<!-- Daniel -->
+  <joint name="imu_joint" type="fixed">
+    <parent link="base_link"/>
+    <child link="imu_link"/>
+    <origin xyz="0.0 0 0.068" rpy="0 0 0"/>
+  </joint>
+  <link name="imu_link"/>
+<!-- Daniel End -->
 <!-- Scan base sensors -->
   <joint name="scan_joint" type="fixed">
@@ -257,5 +265,5 @@
       <origin xyz="0 0 0 " rpy="1.6 0 0"/>
       <geometry>
-        <mesh filename="$(find robot_description)/meshes/kinet.STL" scale="0.001 0.001 0.001"/>
+        <mesh filename="$(find robot_description)/meshes/kinet.STL" scale="0.0001 0.0001 0.0001"/>
       </geometry>
       <material name="${base_color}"/>
