Commit message: Update camera parameters

File: robot_description/urdf/robot.gazebo.macro.xacro (robot description, xacro)
@@ -146,6 +146,6 @@
 <!--              <width>640</width>-->
 <!--              <height>480</height>-->
-             <width>1680</width>
-              <height>1050</height>
+             <width>680</width>
+              <height>480</height>
               <format>R8G8B8</format>
           </image>

File: robot_description/urdf/robot.urdf.xacro (robot description, xacro)
@@ -185,5 +185,5 @@
   </link>
   <joint name="camera_rgb_joint" type="fixed">
-    <origin xyz="0.003 0.011 0.6" rpy="0 0.6 0"/>  <!--<origin xyz="0.003 0.011 0.009" rpy="0 0 0"/> -->
+    <origin xyz="0.003 0.011 0.45" rpy="0 0.6 0"/>  <!--<origin xyz="0.003 0.011 0.009" rpy="0 0 0"/> -->
     <parent link="camera_link"/>
     <child link="camera_rgb_frame"/>
