Commit message: some alteration for nwr model

File: robot_description/urdf/Skid_steering_drive.xacro (robot description, xacro)
@@ -9,6 +9,6 @@
       <leftRearJoint>wheel_left_joint</leftRearJoint>
       <rightRearJoint>wheel_right_joint</rightRearJoint>
-      <wheelSeparation>0.243</wheelSeparation>
-      <wheelDiameter>0.124</wheelDiameter>
+      <wheelSeparation>0.400</wheelSeparation>
+      <wheelDiameter>0.125</wheelDiameter>
       <robotBaseFrame>base_link</robotBaseFrame>
       <torque>20</torque>

File: robot_description/urdf/robot_final.gazebo.macro.xacro (robot description, xacro)
@@ -2,5 +2,5 @@
 <robot name="robot_gaz" xmlns:xacro="http://ros.org/wiki/xacro">
   <!-- <xacro:include filename="$(find robot_description)/urdf/Skid_steering_drive.xacro"/> -->
-  <xacro:include filename="$(find robot_description)/urdf/ros_diff_drive.gazebo.xacro"/>
+  <!-- <xacro:include filename="$(find robot_description)/urdf/ros_diff_drive.gazebo.xacro"/> -->
 <!--  <xacro:include filename="$(find p_g5_description)/urdf/ros_control.gazebo.xacro"/>-->
   <xacro:arg name="laser_visual"  default="false"/>
@@ -8,44 +8,77 @@
   <xacro:arg name="imu_visual"    default="false"/>
   <gazebo reference="base_link">
-    <material>Gazebo/${base_color}</material>
+    <!-- <material>Gazebo/${base_color}</material> -->
+    <material>Gazebo/${player_color}</material>
   </gazebo>
   <gazebo reference="wheel_left_link">
-    <mu1>0.1</mu1>
-    <mu2>0.1</mu2>
-    <kp>500000.0</kp>
-    <kd>10000.0</kd>
-    <minDepth>0.001</minDepth>
-    <maxVel>0.1</maxVel>
-    <fdir1>1 0 0</fdir1>
+    <!-- <mu1>0.7</mu1>
+    <mu2>0.7</mu2>
+    <kp>100000000.0</kp>
+    <kd>1.0</kd>
+    <minDepth>0.01</minDepth>
+    <maxVel>0.1</maxVel>
+    <fdir1>1 0 0</fdir1>
+    <maxVel>10</maxVel> -->
+    <mu1>0.9</mu1>
+    <mu2>0.9</mu2>
+    <kp>1000000.0</kp>
+    <kd>10.0</kd>
+    <minDepth>0.001</minDepth>
+    <maxContacts>1</maxContacts>
+    <fdir1>0 1 0</fdir1>
     <material>Gazebo/${player_color}</material>
   </gazebo>
   <gazebo reference="wheel_left_front_link">
-    <mu1>0</mu1>
-    <mu2>0</mu2>
-    <!-- <kp>500000.0</kp>
-    <kd>10000.0</kd>
-    <minDepth>0.001</minDepth>
-    <maxVel>0.1</maxVel>
-    <fdir1>1 0 0</fdir1> -->
+    <!-- <mu1>0.7</mu1>
+    <mu2>0.7</mu2>
+    <kp>100000000.0</kp>
+    <kd>1.0</kd>
+    <minDepth>0.01</minDepth>
+    <maxVel>0.1</maxVel>
+    <fdir1>1 0 0</fdir1>
+    <maxVel>10</maxVel> -->
+   <mu1>0.9</mu1>
+    <mu2>0.9</mu2>
+    <kp>1000000.0</kp>
+    <kd>10.0</kd>
+    <minDepth>0.001</minDepth>
+    <maxContacts>1</maxContacts>
+    <fdir1>0 1 0</fdir1>
     <material>Gazebo/${player_color}</material>
   </gazebo>
   <gazebo reference="wheel_right_link">
-    <mu1>0.1</mu1>
-    <mu2>0.1</mu2>
-    <kp>500000.0</kp>
-    <kd>10000.0</kd>
-    <minDepth>0.001</minDepth>
-    <maxVel>0.1</maxVel>
-    <fdir1>1 0 0</fdir1>
+    <!-- <mu1>0.7</mu1>
+    <mu2>0.7</mu2>
+    <kp>100000000.0</kp>
+    <kd>1.0</kd>
+    <minDepth>0.01</minDepth>
+    <maxVel>0.1</maxVel>
+    <fdir1>1 0 0</fdir1>
+    <maxVel>10</maxVel> -->
+   <mu1>0.9</mu1>
+    <mu2>0.9</mu2>
+    <kp>1000000.0</kp>
+    <kd>10.0</kd>
+    <minDepth>0.001</minDepth>
+    <maxContacts>1</maxContacts>
+    <fdir1>0 1 0</fdir1>
    <material>Gazebo/${player_color}</material>
   </gazebo>
   <gazebo reference="wheel_right_front_link">
-    <mu1>0</mu1>
-    <mu2>0</mu2>
-    <!-- <kp>500000.0</kp>
-    <kd>10000.0</kd>
-    <minDepth>0.001</minDepth>
-    <maxVel>0.1</maxVel>
-    <fdir1>1 0 0</fdir1> -->
+    <!-- <mu1>0.7</mu1>
+    <mu2>0.7</mu2>
+    <kp>100000000.0</kp>
+    <kd>1.0</kd>
+    <minDepth>0.01</minDepth>
+    <maxVel>0.1</maxVel>
+    <fdir1>1 0 0</fdir1>
+    <maxVel>10</maxVel> -->
+   <mu1>0.9</mu1>
+    <mu2>0.9</mu2>
+    <kp>1000000.0</kp>
+    <kd>10.0</kd>
+    <minDepth>0.001</minDepth>
+    <maxContacts>1</maxContacts>
+    <fdir1>0 1 0</fdir1>
     <material>Gazebo/${player_color}</material>
   </gazebo>
@@ -75,5 +108,5 @@
     <material>Gazebo/Grey</material>
   </gazebo>
-  <gazebo>
+  <!-- <gazebo>
     <plugin name="turtlebot3_waffle_pi_controller" filename="libgazebo_ros_diff_drive.so">
       <commandTopic>cmd_vel</commandTopic>
@@ -95,4 +128,41 @@
       <wheelTorque>10</wheelTorque>
       <rosDebugLevel>na</rosDebugLevel>
+    </plugin>
+  </gazebo> -->
+  <gazebo>
+    <plugin name="SkidSteerDrivePlugin" filename="libgazebo_ros_skid_steer_drive.so">
+      <updateRate>100.0</updateRate>
+      <robotNamespace>robot</robotNamespace>
+      <leftFrontJoint>wheel_left_front_joint</leftFrontJoint>
+      <rightFrontJoint>wheel_right_front_joint</rightFrontJoint>
+      <leftRearJoint>wheel_left_joint</leftRearJoint>
+      <rightRearJoint>wheel_right_joint</rightRearJoint>
+      <wheelSeparation>0.245</wheelSeparation>
+      <wheelDiameter>0.125</wheelDiameter>
+      <robotBaseFrame>base_link</robotBaseFrame>
+      <torque>2</torque>
+      <topicName>cmd_vel</topicName>
+      <broadcastTF>false</broadcastTF>
+      <commandTopic>cmd_vel</commandTopic>
+      <odometryTopic>odom</odometryTopic>
+      <odometryFrame>odom</odometryFrame>
+      <covariance_x>0.0001</covariance_x>
+      <covariance_y>0.0001</covariance_y>
+      <covariance_yaw>0.0001</covariance_yaw>
+        <!-- <dds_domain_id>0</dds_domain_id>
+    <topic_name_twist>cmd_vel</topic_name_twist>
+    <topic_name_odometry>odom</topic_name_odometry>
+    <topic_name_joint>joint</topic_name_joint>
+    <right_front_joint>wheel_right_front_joint</right_front_joint>
+    <right_rear_joint>wheel_right_joint</right_rear_joint>
+    <left_front_joint>wheel_left_front_joint</left_front_joint>
+    <left_rear_joint>wheel_left_joint</left_rear_joint>
+    <wheel_separation>0.4</wheel_separation>
+    <wheel_diameter>0.0625</wheel_diameter>
+    <wheel_torque>5.0</wheel_torque>
+    <update_rate>2</update_rate>
+    <covariance_x>0.0001</covariance_x>
+    <covariance_y>0.0001</covariance_y>
+    <covariance_yaw>0.01</covariance_yaw> -->
     </plugin>
   </gazebo>

File: robot_description/urdf/robot_final.urdf.xacro (robot description, xacro)
@@ -17,24 +17,26 @@
     <parent link="base_footprint"/>
     <child link="base_link" />
-    <origin xyz="0 0 0.0624" rpy="0 0 0"/>
+    <origin xyz="0 0 0.200" rpy="0 0 0"/>
   </joint>
   <link name="base_link">
     <visual>
       <!-- <origin xyz="-0.064 0 0.0" rpy="0 0 0"/> -->
-      <origin xyz="0 0 0" rpy="1.57 0 0"/>
+      <origin xyz="-0.55 -0.175 -0.150" rpy="0 0 0"/>
       <geometry>
         <!-- <mesh filename="package://turtlebot3_description/meshes/bases/waffle_pi_base.stl" scale="0.001 0.001 0.001"/> -->
-        <mesh filename="$(find robot_description)/meshes/base_link.STL" scale="0.001 0.001 0.001"/>
-      </geometry>
-      <material name="${base_color}"/>
-    </visual>
-    <collision>
-      <origin xyz="0.162 -0.125 0.020" rpy="0 0 0"/>
-      <geometry>
-        <box size="0.32 0.16 0.040"/>
-      </geometry>
-    </collision>
-    <inertial>
-      <origin xyz="0.162 -0.1315 0.020" rpy="0 0 0"/>
+        <!-- <mesh filename="$(find robot_description)/meshes/base_link.STL" scale="0.001 0.001 0.001"/> -->
+        <mesh filename="$(find robot_description)/meshes/CarroSemRodasZ.STL" scale="0.001 0.001 0.001 "/>
+        <!-- <mesh filename="$(find robot_description)/meshes/CarroSemRodasZSemKinectics.STL" scale="0.001 0.001 0.001 "/> -->
+      </geometry>
+      <material name="${player_color}"/>
+    </visual>
+    <collision>
+      <origin xyz="-0.250 0 0.222" rpy="0 0 0"/>
+      <geometry>
+        <box size="0.600 0.350 0.480"/>
+      </geometry>
+    </collision>
+    <inertial>
+      <origin xyz="-0.250 0 0.172" rpy="0 0 0"/>
       <mass value="1.3729096e+00"/>
       <inertia ixx="8.7002718e-03" ixy="-4.7576583e-05" ixz="1.1160499e-04"
@@ -43,27 +45,28 @@
     </inertial>
   </link>
+  <!-- wheel_left_joint -->
   <joint name="wheel_left_joint" type="continuous">
     <parent link="base_link"/>
     <child link="wheel_left_link"/>
-    <origin xyz="0.0124 0.0 0.0123" rpy="0 0 0"/>
+    <origin xyz="-0.400 0.1225 -0.1375" rpy="0 0 0"/>
     <axis xyz="0 1 0"/>
   </joint>
   <link name="wheel_left_link">
     <visual>
-      <origin xyz="-0.0624 0 -0.0624" rpy="1.57 0 0"/>
-      <geometry>
-        <mesh filename="$(find robot_description)/meshes/Wheel.STL" scale="0.001 0.001 0.001"/>
-      </geometry>
-      <material name="${player_color}"/>
-    </visual>
-    <collision>
-      <origin xyz="0 -0.0215 0" rpy="1.57 0 0"/>
-      <geometry>
-        <cylinder length="0.045" radius="0.0624"/>
-      </geometry>
-    </collision>
-    <inertial>
-      <origin xyz="0.0 -0.0225 0.0124 " />
-      <mass value="2.8498940e-02" />
+      <origin xyz="0.0625 0 -0.0625" rpy="0 0 3.14"/>
+      <geometry>
+        <mesh filename="$(find robot_description)/meshes/RodaPecaCanto.STL" scale="0.001 0.001 0.001"/>
+      </geometry>
+      <material name="${player_color}"/>
+    </visual>
+    <collision>
+      <origin xyz="0 -0.0215 0" rpy="1.57 0 0"/>
+      <geometry>
+        <cylinder length="0.045" radius="0.0625"/>
+      </geometry>
+    </collision>
+    <inertial>
+      <origin xyz="0 -0.0215 0" rpy="1.57 0 0"/>
+      <mass value="0.5" />
       <inertia ixx="1.1175580e-05" ixy="-4.2369783e-11" ixz="-5.9381719e-09"
                iyy="1.1192413e-05" iyz="-1.4400107e-11"
@@ -75,24 +78,24 @@
     <parent link="base_link"/>
     <child link="wheel_left_front_link"/>
-    <origin xyz="0.3124 0.0 0.0123" rpy="0 0 0"/>
+    <origin xyz="-0.100 0.1225 -0.1375" rpy="0 0 0"/>
     <axis xyz="0 1 0"/>
   </joint>
   <link name="wheel_left_front_link">
     <visual>
-      <origin xyz="-0.0624 0 -0.0624" rpy="1.57 0 0"/>
-      <geometry>
-        <mesh filename="$(find robot_description)/meshes/Wheel.STL" scale="0.001 0.001 0.001"/>
-      </geometry>
-      <material name="${player_color}"/>
-    </visual>
-    <collision>
-      <origin xyz="0 -0.0215 0" rpy="1.57 0 0"/>
-      <geometry>
-        <cylinder length="0.045" radius="0.0624"/>
-      </geometry>
-    </collision>
-    <inertial>
-      <origin xyz="0.0 -0.0225 0.0124 " />
-      <mass value="2.8498940e-02" />
+      <origin xyz="0.0625 0 -0.0625" rpy="0 0 3.14"/>
+      <geometry>
+        <mesh filename="$(find robot_description)/meshes/RodaPecaCanto.STL" scale="0.001 0.001 0.001"/>
+      </geometry>
+      <material name="${player_color}"/>
+    </visual>
+    <collision>
+      <origin xyz="0 -0.0215 0" rpy="1.57 0 0"/>
+      <geometry>
+        <cylinder length="0.045" radius="0.0625"/>
+      </geometry>
+    </collision>
+    <inertial>
+      <origin xyz="0 -0.0215 0" rpy="1.57 0 0"/>
+      <mass value="0.5" />
       <inertia ixx="1.1175580e-05" ixy="-4.2369783e-11" ixz="-5.9381719e-09"
                iyy="1.1192413e-05" iyz="-1.4400107e-11"
@@ -104,24 +107,24 @@
     <parent link="base_link"/>
     <child link="wheel_right_link"/>
-    <origin xyz="0.0124 -0.251 0.0123" rpy="0 0 0"/>
+    <origin xyz="-0.400 -0.1225 -0.1375" rpy="0 0 0"/>
     <axis xyz="0 1 0"/>
   </joint>
   <link name="wheel_right_link">
     <visual>
-      <origin xyz="0.0624 0 -0.0624" rpy="1.57 0 3.14"/>
-      <geometry>
-        <mesh filename="$(find robot_description)/meshes/Wheel.STL" scale="0.001 0.001 0.001"/>
-      </geometry>
-      <material name="${player_color}"/>
-    </visual>
-    <collision>
-      <origin xyz="0 0.0215 0" rpy="1.57 0 0"/>
-      <geometry>
-        <cylinder length="0.045" radius="0.0624"/>
-      </geometry>
-    </collision>
-    <inertial>
-      <origin xyz="0.0 -0.0225 0.0124 " />
-      <mass value="2.8498940e-02" />
+      <origin xyz="-0.0625 0 -0.0625" rpy="0 0 0"/>
+      <geometry>
+        <mesh filename="$(find robot_description)/meshes/RodaPecaCanto.STL" scale="0.001 0.001 0.001"/>
+      </geometry>
+      <material name="${player_color}"/>
+    </visual>
+    <collision>
+      <origin xyz="0 0.0235 0" rpy="1.57 0 0"/>
+      <geometry>
+        <cylinder length="0.045" radius="0.0625"/>
+      </geometry>
+    </collision>
+    <inertial>
+      <origin xyz="0 0.0235 0" rpy="1.57 0 0"/>
+      <mass value="0.5" />
       <inertia ixx="1.1175580e-05" ixy="-4.2369783e-11" ixz="-5.9381719e-09"
                iyy="1.1192413e-05" iyz="-1.4400107e-11"
@@ -131,31 +134,31 @@
   <!-- wheel_right_front_joint -->
  <joint name="wheel_right_front_joint" type="continuous">
-  <parent link="base_link"/>
-  <child link="wheel_right_front_link"/>
-  <origin xyz="0.3124 -0.251 0.0123" rpy="0 0 0"/>
-  <axis xyz="0 1 0"/>
-</joint>
-<link name="wheel_right_front_link">
-  <visual>
-    <origin xyz="0.0624 0 -0.0624" rpy="1.57 0 3.14"/>
-    <geometry>
-      <mesh filename="$(find robot_description)/meshes/Wheel.STL" scale="0.001 0.001 0.001"/>
-    </geometry>
-    <material name="${player_color}"/>
-  </visual>
-  <collision>
-    <origin xyz="0 0.0215 0" rpy="1.57 0 0"/>
-    <geometry>
-      <cylinder length="0.045" radius="0.0624"/>
-    </geometry>
-  </collision>
-  <inertial>
-    <origin xyz="0.0 -0.0225 0.0124 " />
-    <mass value="2.8498940e-02" />
-    <inertia ixx="1.1175580e-05" ixy="-4.2369783e-11" ixz="-5.9381719e-09"
-             iyy="1.1192413e-05" iyz="-1.4400107e-11"
-             izz="2.0712558e-05" />
-    </inertial>
-</link>
+    <parent link="base_link"/>
+    <child link="wheel_right_front_link"/>
+    <origin xyz="-0.100 -0.1225 -0.1375" rpy="0 0 0"/>
+    <axis xyz="0 1 0"/>
+  </joint>
+  <link name="wheel_right_front_link">
+    <visual>
+      <origin xyz="-0.0625 0 -0.0625" rpy="0 0 0"/>
+      <geometry>
+        <mesh filename="$(find robot_description)/meshes/RodaPecaCanto.STL" scale="0.001 0.001 0.001"/>
+      </geometry>
+      <material name="${player_color}"/>
+    </visual>
+    <collision>
+      <origin xyz="0 0.0235 0" rpy="1.57 0 0"/>
+      <geometry>
+        <cylinder length="0.045" radius="0.0625"/>
+      </geometry>
+    </collision>
+    <inertial>
+      <origin xyz="0 0.0235 0" rpy="1.57 0 0"/>
+      <mass value="0.5" />
+      <inertia ixx="1.1175580e-05" ixy="-4.2369783e-11" ixz="-5.9381719e-09"
+               iyy="1.1192413e-05" iyz="-1.4400107e-11"
+               izz="2.0712558e-05" />
+      </inertial>
+  </link>
 <!--
   <joint name="caster_back_right_joint" type="fixed">
@@ -219,5 +222,5 @@
 <!-- Daniel End -->
 <!-- Scan base sensors -->
-  <joint name="scan_joint" type="fixed">
+  <!-- <joint name="scan_joint" type="fixed">
     <parent link="base_link"/>
     <child link="base_scan"/>
@@ -228,5 +231,5 @@
       <origin xyz="-0.136 0.0289 -0.025" rpy="1.57 0 0"/>
       <geometry>
-        <mesh filename="$(find robot_description)/meshes/base_scan_sensors.STL" scale="0.001 0.001 0.001"/>
+        <mesh filename="$(find robot_description)/meshes/Portico_1 - portico2-1.STL" scale="0.001 0.001 0.001"/>
       </geometry>
       <material name="${player_color}"/>
@@ -245,8 +248,8 @@
                izz="0.001" />
     </inertial>
-  </link>
+  </link>  -->
   <!-- Camera link -->
   <joint name="camera_joint" type="fixed">
-    <origin xyz="0.073 -0.011 0.084" rpy="0 0 0"/>
+    <origin xyz="-0.05 0 0.350" rpy="0 0 0"/>
     <parent link="base_link"/>
     <child link="camera_link"/>
@@ -256,6 +259,5 @@
   <!-- camera_rgb_joint -->
   <joint name="camera_rgb_joint" type="fixed">
-    <!-- <origin xyz="0.003 0.011 0.6" rpy="0 0.6 0"/>     -->
-    <origin xyz="0.3 0.011 0.45" rpy="0 0.6 0"/>
+    <origin xyz="0 0 0" rpy="0 0 0"/>
     <parent link="camera_link"/>
     <child link="camera_rgb_frame"/>
@@ -263,7 +265,7 @@
   <link name="camera_rgb_frame">
     <visual>
-      <origin xyz="0 0 0 " rpy="1.6 0 0"/>
-      <geometry>
-        <mesh filename="$(find robot_description)/meshes/kinet.STL" scale="0.0001 0.0001 0.0001"/>
+      <origin xyz="0.03 -0.138 -0.05 " rpy="0 0 1.57"/>
+      <geometry>
+        <mesh filename="$(find robot_description)/meshes/KinectZ.STL" scale="0.001 0.001 0.001"/>
       </geometry>
       <material name="${base_color}"/>
@@ -277,9 +279,9 @@
       </link>
   <!-- camera_rgb_optical_joint -->
-  <!-- <joint name="camera_rgb_optical_joint" type="fixed">
+  <joint name="camera_rgb_optical_joint" type="fixed">
     <origin xyz="0 0 0" rpy="-1.57 0 -1.57"/>
     <parent link="camera_rgb_frame"/>
     <child link="camera_rgb_optical_frame"/>
   </joint>
-  <link name="camera_rgb_optical_frame"/>  -->
+  <link name="camera_rgb_optical_frame"/>
 </robot>
