Commit message: Upload more images for height and angle

File: robot_description/urdf/robot.urdf.xacro (robot description, xacro)
@@ -185,5 +185,5 @@
   </link>
   <joint name="camera_rgb_joint" type="fixed">
-    <origin xyz="0.003 0.011 0.009" rpy="0 0 0"/>
+     <origin xyz="0.003 0.011 0.009" rpy="0 0 0"/>  <!--<origin xyz="0.003 0.011 0.009" rpy="0 0 0"/> -->
     <parent link="camera_link"/>
     <child link="camera_rgb_frame"/>

File: robot_description/urdf/robot_final.urdf.xacro (robot description, xacro)
@@ -250,5 +250,5 @@
   </link>
   <joint name="camera_rgb_joint" type="fixed">
-   <origin xyz="0.003 0.011 0.6" rpy="0 0 0"/>       <!-- old values (SF):xyz="0.003 0.011 0.6" rpy="0 0.6 0"-->
+    <origin xyz="0.003 0.011 0.45" rpy="0 0.15 0"/>    -  <!-- old values (SF):xyz="0.003 0.011 0.6" rpy="0 0.6 0"-->
     <parent link="camera_link"/>
     <child link="camera_rgb_frame"/>

Commit message: spaw do turtlebot

File: robot_description/urdf/robot.urdf.xacro (robot description, xacro)
@@ -185,5 +185,5 @@
   </link>
   <joint name="camera_rgb_joint" type="fixed">
-     <origin xyz="0.003 0.011 0.009" rpy="0 0 0"/>  <!--<origin xyz="0.003 0.011 0.009" rpy="0 0 0"/> -->
+    <origin xyz="0.003 0.011 0.6" rpy="0 0.6 0"/>  <!--<origin xyz="0.003 0.011 0.009" rpy="0 0 0"/> -->
     <parent link="camera_link"/>
     <child link="camera_rgb_frame"/>

Commit message: Update write_csv2.py

File: robot_description/urdf/robot.urdf.xacro (robot description, xacro)
@@ -185,5 +185,5 @@
   </link>
   <joint name="camera_rgb_joint" type="fixed">
-    <origin xyz="0.003 0.011 0.45" rpy="0 0.6 0"/>  <!--<origin xyz="0.003 0.011 0.009" rpy="0 0 0"/> -->
+    <origin xyz="0.003 0.011 0.59" rpy="0 0.6 0"/>  <!--<origin xyz="0.003 0.011 0.009" rpy="0 0 0"/> -->
     <parent link="camera_link"/>
     <child link="camera_rgb_frame"/>

Commit message: back to 0.45 height

File: robot_description/urdf/robot.urdf.xacro (robot description, xacro)
@@ -185,5 +185,5 @@
   </link>
   <joint name="camera_rgb_joint" type="fixed">
-    <origin xyz="0.003 0.011 0.59" rpy="0 0.6 0"/>  <!--<origin xyz="0.003 0.011 0.009" rpy="0 0 0"/> -->
+    <origin xyz="0.003 0.011 0.45" rpy="0 0.6 0"/>  <!--<origin xyz="0.003 0.011 0.009" rpy="0 0 0"/> -->
     <parent link="camera_link"/>
     <child link="camera_rgb_frame"/>

Commit message: Upload write csv for cnn model

File: robot_description/urdf/robot.urdf.xacro (robot description, xacro)
@@ -185,5 +185,5 @@
   </link>
   <joint name="camera_rgb_joint" type="fixed">
-    <origin xyz="0.003 0.011 0.45" rpy="0 0.6 0"/>  <!--<origin xyz="0.003 0.011 0.009" rpy="0 0 0"/> -->
+    <origin xyz="0.003 0.011 0.45" rpy="0 0.6 0"/>  <!--<origin xyz="0.003 0.011 0.009" rpy="0 0 0"/> --> <!--<origin xyz="0.003 0.011 0.59" rpy="0 0.4 0"/> -->
     <parent link="camera_link"/>
     <child link="camera_rgb_frame"/>

Commit message: improv CNN

File: robot_description/urdf/robot.urdf.xacro (robot description, xacro)
@@ -185,5 +185,5 @@
   </link>
   <joint name="camera_rgb_joint" type="fixed">
-    <origin xyz="0.003 0.011 0.45" rpy="0 0.6 0"/>  <!--<origin xyz="0.003 0.011 0.009" rpy="0 0 0"/> --> <!--<origin xyz="0.003 0.011 0.59" rpy="0 0.4 0"/> -->
+    <origin xyz="0.003 0.011 0.59" rpy="0 0.4 0"/>  <!--<origin xyz="0.003 0.011 0.009" rpy="0 0 0"/> --> <!--<origin xyz="0.003 0.011 0.45" rpy="0 0.6 0"/> -->
     <parent link="camera_link"/>
     <child link="camera_rgb_frame"/>
