Commit message: Merge branch 'dev' of https://github.com/DanielCoelho112/AutoMec-AD into dev

File: ackermann_vehicle_description/urdf/robot02.urdf.xacro (robot description, xacro)
@@ -54,8 +54,12 @@
        is a "zero offset" wheel. hex_hub_depth = tire_width / 2 -
        axle_length. -->
-  <xacro:property name="hub_dia" value="0.09652"/>
-  <xacro:property name="tire_dia" value="0.14605"/>
-  <xacro:property name="tire_width" value="0.0889"/>
-  <xacro:property name="hex_hub_depth" value="0.01445"/>
+  <!-- <xacro:property name="hub_dia" value="0.09652"/> -->
+  <xacro:property name="hub_dia" value="0.0826"/>
+  <!-- <xacro:property name="tire_dia" value="0.14605"/> -->
+  <xacro:property name="tire_dia" value="0.125"/>
+  <!-- <xacro:property name="tire_width" value="0.0889"/> -->
+  <xacro:property name="tire_width" value="0.045"/>
+  <!-- <xacro:property name="hex_hub_depth" value="0.01445"/> -->
+  <xacro:property name="hex_hub_depth" value="-0.0075"/>
   <xacro:property name="wheel_mass" value="0.29"/>
   <!-- hex_hub_dist is the distance between left and right hex hubs when
@@ -63,6 +67,8 @@
        from a U joint to the corresponding hex hub. wheel_travel is the
        vertical wheel travel. -->
-  <xacro:property name="wheelbase" value="0.335"/>
-  <xacro:property name="hex_hub_dist" value="0.365"/>
+  <!-- <xacro:property name="wheelbase" value="0.335"/> -->
+  <xacro:property name="wheelbase" value="0.245"/>
+  <!-- <xacro:property name="hex_hub_dist" value="0.365"/> -->
+  <xacro:property name="hex_hub_dist" value="0.27"/>
   <xacro:property name="axle_length" value="0.03"/>
   <xacro:property name="wheel_travel" value="0.084"/>
@@ -242,10 +248,12 @@
     <link name="${lr_prefix}_${fr_prefix}_wheel">
       <visual>
-        <origin xyz="0
+        <!-- <origin xyz="0
                      ${lr_reflect * (axle_length - (tire_width /
                      2 - hex_hub_depth))}
-                     0"/>
+                     0" /> -->
+        <origin xyz="-0.0825 0.0625 0" rpy="1.57 0 0"/>
         <geometry>
-          <cylinder radius="${tire_dia / 2}" length="${tire_width}"/>
+          <!--<cylinder radius="${tire_dia / 2}" length="${tire_width}"/>-->
+          <mesh filename="$(find robot_description)/meshes/RodaPecaCanto.STL" scale="0.001 0.001 0.001"/>
         </geometry>
         <material name="tire_mat"/>
@@ -322,7 +330,9 @@
   <link name="chassis">
     <visual>
-      <origin xyz="0 0 ${-chassis_height / 2}"/>
-      <geometry>
-        <box size="${chassis_length} ${chassis_width} ${chassis_height}"/>
+      <!-- <origin xyz="0 0 ${-chassis_height / 2}"/> -->
+      <origin xyz="-0.3 -0.195  -0.045"/> <!--x z y-->
+      <geometry>
+        <!-- <box size="${chassis_length} ${chassis_width} ${chassis_height}"/> -->
+        <mesh filename="$(find robot_description)/meshes/CarroSemRodasZ.STL" scale="0.001 0.001 0.001 "/>
       </geometry>
       <material name="chassis_mat"/>

Commit message: Camera and screen dimensions changes, added the undistorted picture to both signal recognitions

File: ackermann_vehicle_description/urdf/robot02.urdf.xacro (robot description, xacro)
@@ -404,5 +404,5 @@
   <link name="camera_rgb_optical_frame"/>
   <joint name="camera2_joint" type="fixed">
-    <origin xyz="0.073 -0.011 0.01" rpy="0 -0.6 0"/>
+    <origin xyz="0.073 -0.011 0.14" rpy="0 0 0"/>
     <parent link="base_link"/>
     <child link="camera2_link"/>
