Commit message: urdf robot04 and launch names

File: traxxas_description/urdf/robot04.gazebo.macro.xacro (robot description, xacro)
@@ -105,3 +105,67 @@
     </sensor>
   </gazebo>
+  <gazebo reference="cameral_rgb_frame">
+    <sensor type="camera" name="Pi Camera">
+      <always_on>true</always_on>
+      <visualize>$(arg camera_visual)</visualize>
+      <camera>
+          <horizontal_fov>1.085595</horizontal_fov>
+          <image>
+             <width>680</width>
+              <height>480</height>
+              <format>R8G8B8</format>
+          </image>
+          <clip>
+              <near>0.03</near>
+              <far>100</far>
+          </clip>
+      </camera>
+      <plugin name="camera_controller" filename="libgazebo_ros_camera.so">
+        <alwaysOn>true</alwaysOn>
+        <updateRate>30.0</updateRate>
+        <cameraName>cameral</cameraName>
+        <frameName>cameral_rgb_optical_frame</frameName>
+        <imageTopicName>rgb/image_raw</imageTopicName>
+        <cameraInfoTopicName>rgb/camera_info</cameraInfoTopicName>
+        <hackBaseline>0.07</hackBaseline>
+        <distortionK1>0.0</distortionK1>
+        <distortionK2>0.0</distortionK2>
+        <distortionK3>0.0</distortionK3>
+        <distortionT1>0.0</distortionT1>
+        <distortionT2>0.0</distortionT2>
+      </plugin>
+    </sensor>
+  </gazebo>
+  <gazebo reference="camerar_rgb_frame">
+    <sensor type="camera" name="Pi Camera">
+      <always_on>true</always_on>
+      <visualize>$(arg camera_visual)</visualize>
+      <camera>
+          <horizontal_fov>1.085595</horizontal_fov>
+          <image>
+             <width>680</width>
+              <height>480</height>
+              <format>R8G8B8</format>
+          </image>
+          <clip>
+              <near>0.03</near>
+              <far>100</far>
+          </clip>
+      </camera>
+      <plugin name="camera_controller" filename="libgazebo_ros_camera.so">
+        <alwaysOn>true</alwaysOn>
+        <updateRate>30.0</updateRate>
+        <cameraName>camerar</cameraName>
+        <frameName>camerar_rgb_optical_frame</frameName>
+        <imageTopicName>rgb/image_raw</imageTopicName>
+        <cameraInfoTopicName>rgb/camera_info</cameraInfoTopicName>
+        <hackBaseline>0.07</hackBaseline>
+        <distortionK1>0.0</distortionK1>
+        <distortionK2>0.0</distortionK2>
+        <distortionK3>0.0</distortionK3>
+        <distortionT1>0.0</distortionT1>
+        <distortionT2>0.0</distortionT2>
+      </plugin>
+    </sensor>
+  </gazebo>
 </robot>

File: traxxas_description/urdf/robot04.urdf.xacro (robot description, xacro)
@@ -27,12 +27,8 @@
        is a "zero offset" wheel. hex_hub_depth = tire_width / 2 -
        axle_length. -->
-  <!-- <xacro:property name="hub_dia" value="0.09652"/> -->
-  <xacro:property name="hub_dia" value="0.0826"/>
-  <!-- <xacro:property name="tire_dia" value="0.14605"/> -->
-  <xacro:property name="tire_dia" value="0.125"/>
-  <!-- <xacro:property name="tire_width" value="0.0889"/> -->
-  <xacro:property name="tire_width" value="0.045"/>
-  <!-- <xacro:property name="hex_hub_depth" value="0.01445"/> -->
-  <xacro:property name="hex_hub_depth" value="-0.0075"/>
+  <xacro:property name="hub_dia" value="0.09652"/>
+  <xacro:property name="tire_dia" value="0.14605"/>
+  <xacro:property name="tire_width" value="0.0889"/>
+  <xacro:property name="hex_hub_depth" value="0.01445"/>
   <xacro:property name="wheel_mass" value="0.29"/>
   <!-- hex_hub_dist is the distance between left and right hex hubs when
@@ -40,8 +36,6 @@
        from a U joint to the corresponding hex hub. wheel_travel is the
        vertical wheel travel. -->
-  <!-- <xacro:property name="wheelbase" value="0.335"/> -->
-  <xacro:property name="wheelbase" value="0.245"/>
-  <!-- <xacro:property name="hex_hub_dist" value="0.365"/> -->
-  <xacro:property name="hex_hub_dist" value="0.27"/>
+  <xacro:property name="wheelbase" value="0.335"/>
+  <xacro:property name="hex_hub_dist" value="0.365"/>
   <xacro:property name="axle_length" value="0.03"/>
   <xacro:property name="wheel_travel" value="0.084"/>
@@ -89,5 +83,5 @@
     <color rgba="0 1 0 1"/>
   </material>
-  <xacro:include filename="$(find traxxas_description)/urdf/robot03.gazebo.macro.xacro"/>
+  <xacro:include filename="$(find traxxas_description)/urdf/robot04.gazebo.macro.xacro"/>
   <!-- Null inertial element. This is needed to make the model work with
        Gazebo. -->
@@ -221,12 +215,10 @@
     <link name="${lr_prefix}_${fr_prefix}_wheel">
       <visual>
-        <!-- <origin xyz="0
+        <origin xyz="0
                      ${lr_reflect * (axle_length - (tire_width /
                      2 - hex_hub_depth))}
-                     0" /> -->
-        <origin xyz="-0.0825 0.0625 0" rpy="1.57 0 0"/>
+                     0"/>
         <geometry>
-          <!--<cylinder radius="${tire_dia / 2}" length="${tire_width}"/>-->
-          <mesh filename="$(find traxxas_description)/meshes/RodaPecaCanto.STL" scale="0.001 0.001 0.001"/>
+          <cylinder radius="${tire_dia / 2}" length="${tire_width}"/>
         </geometry>
         <material name="tire_mat"/>
@@ -303,9 +295,7 @@
   <link name="chassis">
     <visual>
-      <!-- <origin xyz="0 0 ${-chassis_height / 2}"/> -->
-      <origin xyz="-0.3 -0.195  -0.045"/> <!--x z y-->
-      <geometry>
-        <!-- <box size="${chassis_length} ${chassis_width} ${chassis_height}"/> -->
-        <mesh filename="$(find traxxas_description)/meshes/CarroSemRodasZ.STL" scale="0.001 0.001 0.001 "/>
+      <origin xyz="0 0 ${-chassis_height / 2}"/>
+      <geometry>
+        <box size="${chassis_length} ${chassis_width} ${chassis_height}"/>
       </geometry>
       <material name="chassis_mat"/>
@@ -355,6 +345,7 @@
     </visual>
   </link>
+  <!--lane camara center -->
   <joint name="camera_joint" type="fixed">
-    <origin xyz="0.073 -0.011 0.084" rpy="0 0.6 0"/>
+    <origin xyz="0.073 0.0 0.084" rpy="0 0.6 0"/>
     <parent link="base_link"/>
     <child link="camera_link"/>
@@ -368,5 +359,5 @@
     </visual>
     <collision>
-      <origin xyz="0.005 0.011 0.013" rpy="0 0 0"/>
+      <origin xyz="0.005 0.0 0.013" rpy="0 0 0"/>
       <geometry>
         <box size="0.015 0.030 0.027"/>
@@ -375,5 +366,5 @@
   </link>
   <joint name="camera_rgb_joint" type="fixed">
-    <origin xyz="0.003 0.011 0.45" rpy="0 0 0"/>
+    <origin xyz="0.003 0.0 0.45" rpy="0 0 0"/>
       <parent link="camera_link"/>
     <child link="camera_rgb_frame"/>
@@ -386,6 +377,7 @@
   </joint>
   <link name="camera_rgb_optical_frame"/>
+  <!--signal camara -->
   <joint name="camera2_joint" type="fixed">
-    <origin xyz="0.073 -0.011 0.01" rpy="0 -0.6 0"/>
+    <origin xyz="0.073 0.0 0.14" rpy="0 0 0"/>
     <parent link="base_link"/>
     <child link="camera2_link"/>
@@ -399,5 +391,5 @@
     </visual>
     <collision>
-      <origin xyz="0.005 0.011 0.013" rpy="0 0 0"/>
+      <origin xyz="0.005 0.0 0.013" rpy="0 0 0"/>
       <geometry>
         <box size="0.015 0.030 0.027"/>
@@ -406,5 +398,5 @@
   </link>
   <joint name="camera2_rgb_joint" type="fixed">
-    <origin xyz="0.003 0.011 0.45" rpy="0 0 0"/>
+    <origin xyz="0.003 0.0 0.45" rpy="0 0 0"/>
     <parent link="camera2_link"/>
     <child link="camera2_rgb_frame"/>
@@ -417,4 +409,69 @@
   </joint>
   <link name="camera2_rgb_optical_frame"/>
+  <!--lane camara left -->
+  <joint name="cameral_joint" type="fixed">
+    <origin xyz="0.073 0.15 0.084" rpy="0 0.6 0"/>
+    <parent link="base_link"/>
+    <child link="cameral_link"/>
+  </joint>
+  <link name="cameral_link">
+    <visual>
+      <geometry>
+        <box size="0.015 0.030 0.027"/>
+      </geometry>
+      <material name="camera_mat"/>
+    </visual>
+    <collision>
+      <origin xyz="0.005 0.011 0.013" rpy="0 0 0"/>
+      <geometry>
+        <box size="0.015 0.030 0.027"/>
+      </geometry>
+    </collision>
+  </link>
+  <joint name="cameral_rgb_joint" type="fixed">
+    <origin xyz="0.003 0.011 0.45" rpy="0 0 0"/>
+      <parent link="cameral_link"/>
+    <child link="cameral_rgb_frame"/>
+  </joint>
+  <link name="cameral_rgb_frame"/>
+  <joint name="cameral_rgb_optical_joint" type="fixed">
+    <origin xyz="0 0 0" rpy="-1.57 0 -1.57"/>
+    <parent link="cameral_rgb_frame"/>
+    <child link="cameral_rgb_optical_frame"/>
+  </joint>
+  <link name="cameral_rgb_optical_frame"/>
+  <!--lane camara right -->
+  <joint name="camerar_joint" type="fixed">
+    <origin xyz="0.073 -0.15 0.084" rpy="0 0.6 0"/>
+    <parent link="base_link"/>
+    <child link="camerar_link"/>
+  </joint>
+  <link name="camerar_link">
+    <visual>
+      <geometry>
+        <box size="0.015 0.030 0.027"/>
+      </geometry>
+      <material name="camera_mat"/>
+    </visual>
+    <collision>
+      <origin xyz="0.005 0.011 0.013" rpy="0 0 0"/>
+      <geometry>
+        <box size="0.015 0.030 0.027"/>
+      </geometry>
+    </collision>
+  </link>
+  <joint name="camerar_rgb_joint" type="fixed">
+    <origin xyz="0.003 0.011 0.45" rpy="0 0 0"/>
+      <parent link="camerar_link"/>
+    <child link="camerar_rgb_frame"/>
+  </joint>
+  <link name="camerar_rgb_frame"/>
+  <joint name="camerar_rgb_optical_joint" type="fixed">
+    <origin xyz="0 0 0" rpy="-1.57 0 -1.57"/>
+    <parent link="camerar_rgb_frame"/>
+    <child link="camerar_rgb_optical_frame"/>
+  </joint>
+  <link name="camerar_rgb_optical_frame"/>
+  <!--gazebo control -->
   <gazebo>
     <plugin name="gazebo_ros_control" filename="libgazebo_ros_control.so">
