Commit message: issue 63, change wheel color to darkgray on gazebo

File: traxxas_description/urdf/robot04.urdf.xacro (robot description, xacro)
@@ -238,5 +238,5 @@
     </link>
     <gazebo reference="${lr_prefix}_${fr_prefix}_wheel">
-      <material>Gazebo/Black</material>
+      <material>Gazebo/DarkGrey</material>
     </gazebo>
   </xacro:macro>

File: traxxas_description/urdf/robot05.urdf.xacro (robot description, xacro)
@@ -238,5 +238,5 @@
     </link>
     <gazebo reference="${lr_prefix}_${fr_prefix}_wheel">
-      <material>Gazebo/Black</material>
+      <material>Gazebo/DarkGrey</material>
     </gazebo>
   </xacro:macro>
