Commit message: issue 41 (wip),  kinect gazebo update

File: traxxas_description/urdf/robot05.gazebo.macro.xacro (robot description, xacro)
@@ -172,5 +172,5 @@
     <sensor name="kinect" type="depth">
         <!-- openni plugin has the x pointing towards the scene, so rotate to have z -->
-        <pose frame="kinect">0.0 0.0 0.0 0.0 -1.5708 1.5708</pose>
+        <pose frame="kinect_place_optical_frame">0.0 0.0 0.0 -1.5708 0.0 1.5708</pose>
         <mesh><uri>file://traxxas_description/meshes/kinect.dae</uri></mesh>
         <camera>
@@ -211,8 +211,6 @@
     </sensor>
 </gazebo>
-<gazebo reference="kinect2_place_optical_frame">
+<gazebo reference="kinect2_optical_frame">
     <sensor name="kinect2" type="depth">
-        <!-- openni plugin has the x pointing towards the scene, so rotate to have z -->
-        <pose frame="world">0.0 0.0 1.0 0.0 -1.5708 1.5708</pose>
         <camera>
             <horizontal_fov>0.74839718</horizontal_fov>
@@ -244,5 +242,5 @@
             <depthImageInfoTopicName>/3d_image2/camera_info</depthImageInfoTopicName>
             <pointCloudTopicName>/3d_image2/3d_cloud</pointCloudTopicName>
-            <frameName>kinect2_place_optical_frame</frameName>
+            <frameName>kinect2_optical_frame</frameName>
             <pointCloudCutoff>0.5</pointCloudCutoff>
             <pointCloudCutoffMax>2.0</pointCloudCutoffMax>

File: traxxas_description/urdf/robot05.urdf.xacro (robot description, xacro)
@@ -355,5 +355,5 @@
       <geometry>
         <box size="0.015 0.030 0.027"/>
-        <mesh filename="package://traxxas_description/meshes/kinect.dae"/>
+        <!-- <mesh filename="package://traxxas_description/meshes/kinect.dae" /> -->
       </geometry>
       <material name="kinect_mat"/>
@@ -380,34 +380,28 @@
   <!--signal camara -->
   <joint name="kinect2_joint" type="fixed">
-    <origin xyz="0.073 0.0 0.14" rpy="0 0 0"/>
+    <origin xyz="0.073 0.0 0.14" rpy="0 0 1.5708"/>
     <parent link="base_link"/>
     <child link="kinect2_link"/>
   </joint>
   <link name="kinect2_link">
-    <visual>
-      <geometry>
-        <box size="0.015 0.030 0.027"/>
-      </geometry>
-      <material name="kinect_mat"/>
+    <origin xyz="0 0 0" rpy="0 0 0"/>
+    <visual>
+      <origin xyz="0 0 0" rpy="0 0 0"/>
+      <geometry>
+        <mesh filename="package://traxxas_description/meshes/kinect.dae"/>
+      </geometry>
     </visual>
     <collision>
-      <origin xyz="0.005 0.0 0.013" rpy="0 0 0"/>
-      <geometry>
-        <box size="0.015 0.030 0.027"/>
+      <geometry>
+        <box size="0.06 0.30 0.07"/>
       </geometry>
     </collision>
   </link>
-  <joint name="kinect2_place_joint" type="fixed">
-    <origin xyz="0.003 0.0 0.45" rpy="0 0 0"/>
+  <joint name="kinect2_optical_joint" type="fixed">
+    <origin xyz="0 0 0" rpy="0 0 -1.5708"/>
     <parent link="kinect2_link"/>
-    <child link="kinect2_place_frame"/>
-  </joint>
-  <link name="kinect2_place_frame"/>
-  <joint name="kinect2_place_optical_joint" type="fixed">
-    <origin xyz="0 0 0" rpy="-1.57 0 -1.57"/>
-    <parent link="kinect2_place_frame"/>
-    <child link="kinect2_place_optical_frame"/>
-  </joint>
-  <link name="kinect2_place_optical_frame"/>
+    <child link="kinect2_optical_frame"/>
+  </joint>
+  <link name="kinect2_optical_frame" />
   <!--lane camara left -->
   <joint name="cameral_joint" type="fixed">

Commit message: issue 41, dual kinect gazebo

File: traxxas_description/urdf/robot05.gazebo.macro.xacro (robot description, xacro)
@@ -169,9 +169,8 @@
     </sensor>
   </gazebo>
-<gazebo reference="kinect_place_optical_frame">
+<gazebo reference="kinect_optical_frame">
     <sensor name="kinect" type="depth">
         <!-- openni plugin has the x pointing towards the scene, so rotate to have z -->
-        <pose frame="kinect_place_optical_frame">0.0 0.0 0.0 -1.5708 0.0 1.5708</pose>
-        <mesh><uri>file://traxxas_description/meshes/kinect.dae</uri></mesh>
+        <pose frame="world">0.0 0.0 0.0 -1.5708 0.0 1.5708</pose>
         <camera>
             <horizontal_fov>0.74839718</horizontal_fov>
@@ -203,5 +202,5 @@
             <depthImageInfoTopicName>/3d_image/camera_info</depthImageInfoTopicName>
             <pointCloudTopicName>/3d_image/3d_cloud</pointCloudTopicName>
-            <frameName>kinect_place_optical_frame</frameName>
+            <frameName>kinect_optical_frame1</frameName>
             <pointCloudCutoff>0.5</pointCloudCutoff>
             <pointCloudCutoffMax>2.0</pointCloudCutoffMax>
@@ -213,4 +212,6 @@
 <gazebo reference="kinect2_optical_frame">
     <sensor name="kinect2" type="depth">
+        <!-- openni plugin has the x pointing towards the scene, so rotate to have z -->
+        <pose frame="world">0.0 0.0 0.0 -1.5708 0.0 1.5708</pose>
         <camera>
             <horizontal_fov>0.74839718</horizontal_fov>
@@ -242,5 +243,5 @@
             <depthImageInfoTopicName>/3d_image2/camera_info</depthImageInfoTopicName>
             <pointCloudTopicName>/3d_image2/3d_cloud</pointCloudTopicName>
-            <frameName>kinect2_optical_frame</frameName>
+            <frameName>kinect2_optical_frame1</frameName>
             <pointCloudCutoff>0.5</pointCloudCutoff>
             <pointCloudCutoffMax>2.0</pointCloudCutoffMax>

File: traxxas_description/urdf/robot05.urdf.xacro (robot description, xacro)
@@ -347,38 +347,31 @@
   <!--lane kinect camara center -->
   <joint name="kinect_joint" type="fixed">
-    <origin xyz="0.073 0.0 0.084" rpy="0 0.6 0"/>
+    <origin xyz="0.073 0.0 0.12" rpy="0.6 0.0 1.5708"/>
     <parent link="base_link"/>
     <child link="kinect_link"/>
   </joint>
   <link name="kinect_link">
-    <visual>
-      <geometry>
-        <box size="0.015 0.030 0.027"/>
-        <!-- <mesh filename="package://traxxas_description/meshes/kinect.dae" /> -->
-      </geometry>
-      <material name="kinect_mat"/>
+    <origin xyz="0 0 0" rpy="0 0 0"/>
+    <visual>
+      <origin xyz="0 0 0" rpy="0 0 0"/>
+      <geometry>
+        <mesh filename="package://traxxas_description/meshes/kinect.dae"/>
+      </geometry>
     </visual>
     <collision>
-      <origin xyz="0.005 0.0 0.013" rpy="0 0 0"/>
-      <geometry>
-        <box size="0.015 0.030 0.027"/>
+      <geometry>
+        <box size="0.06 0.30 0.07"/>
       </geometry>
     </collision>
   </link>
-  <joint name="kinect_place_joint" type="fixed">
-    <origin xyz="0.003 0.0 0.45" rpy="0 0 0"/>
+  <joint name="kinect_optical_joint" type="fixed">
+    <origin xyz="0 0 0" rpy="0 0 -1.5708"/>
     <parent link="kinect_link"/>
-    <child link="kinect_place_frame"/>
-  </joint>
-  <link name="kinect_place_frame"/>
-  <joint name="kinect_place_optical_joint" type="fixed">
-    <origin xyz="0 0 0" rpy="-1.57 0 -1.57"/>
-    <parent link="kinect_place_frame"/>
-    <child link="kinect_place_optical_frame"/>
-  </joint>
-  <link name="kinect_place_optical_frame"/>
-  <!--signal camara -->
+    <child link="kinect_optical_frame"/>
+  </joint>
+  <link name="kinect_optical_frame"/>
+  <!--signal kinect camara -->
   <joint name="kinect2_joint" type="fixed">
-    <origin xyz="0.073 0.0 0.14" rpy="0 0 1.5708"/>
+    <origin xyz="0.073 0.0 0.24" rpy="0 0 1.5708"/>
     <parent link="base_link"/>
     <child link="kinect2_link"/>

Commit message: urdf models update

File: traxxas_description/urdf/robot05.gazebo.macro.xacro (robot description, xacro)
@@ -169,3 +169,85 @@
     </sensor>
   </gazebo>
+<gazebo reference="kinect_optical_frame">
+    <sensor name="kinect" type="depth">
+        <!-- openni plugin has the x pointing towards the scene, so rotate to have z -->
+        <pose frame="world">0.0 0.0 0.0 -1.5708 0.0 1.5708</pose>
+        <camera>
+            <horizontal_fov>0.74839718</horizontal_fov>
+            <image>
+                <width>1280</width>
+                <height>1024</height>
+                <format>L_INT8</format>
+            </image>
+            <clip>
+                <near>0.1</near>
+                <far>10.0</far>
+            </clip>
+            <noise>
+                <type>gaussian</type>
+                <mean>0.5</mean>
+                <stddev>1.0</stddev>
+            </noise>
+        </camera>
+        <plugin name="kinect_plugin" filename="libgazebo_ros_openni_kinect.so">
+            <baseline>0.1</baseline>
+            <alwaysOn>true</alwaysOn>
+            <!-- Keep this zero, update_rate in the parent <sensor> tag
+            will control the frame rate. -->
+            <updateRate>0.0</updateRate>
+            <cameraName>kinect_test</cameraName>
+            <imageTopicName>/3d_image/image_raw</imageTopicName>
+            <cameraInfoTopicName>/3d_image/camera_info</cameraInfoTopicName>
+            <depthImageTopicName>/3d_image/image_raw_depth</depthImageTopicName>
+            <depthImageInfoTopicName>/3d_image/camera_info</depthImageInfoTopicName>
+            <pointCloudTopicName>/3d_image/3d_cloud</pointCloudTopicName>
+            <frameName>kinect_optical_frame1</frameName>
+            <pointCloudCutoff>0.5</pointCloudCutoff>
+            <pointCloudCutoffMax>2.0</pointCloudCutoffMax>
+        </plugin>
+        <always_on>true</always_on>
+        <update_rate>1.0</update_rate>
+    </sensor>
+</gazebo>
+<gazebo reference="kinect2_optical_frame">
+    <sensor name="kinect2" type="depth">
+        <!-- openni plugin has the x pointing towards the scene, so rotate to have z -->
+        <pose frame="world">0.0 0.0 0.0 -1.5708 0.0 1.5708</pose>
+        <camera>
+            <horizontal_fov>0.74839718</horizontal_fov>
+            <image>
+                <width>1280</width>
+                <height>1024</height>
+                <format>L_INT8</format>
+            </image>
+            <clip>
+                <near>0.1</near>
+                <far>10.0</far>
+            </clip>
+            <noise>
+                <type>gaussian</type>
+                <mean>0.5</mean>
+                <stddev>1.0</stddev>
+            </noise>
+        </camera>
+        <plugin name="kinect_plugin" filename="libgazebo_ros_openni_kinect.so">
+            <baseline>0.1</baseline>
+            <alwaysOn>true</alwaysOn>
+            <!-- Keep this zero, update_rate in the parent <sensor> tag
+            will control the frame rate. -->
+            <updateRate>0.0</updateRate>
+            <cameraName>kinect_test2</cameraName>
+            <imageTopicName>/3d_image2/image_raw</imageTopicName>
+            <cameraInfoTopicName>/3d_image2/camera_info</cameraInfoTopicName>
+            <depthImageTopicName>/3d_image2/image_raw_depth</depthImageTopicName>
+            <depthImageInfoTopicName>/3d_image2/camera_info</depthImageInfoTopicName>
+            <pointCloudTopicName>/3d_image2/3d_cloud</pointCloudTopicName>
+            <frameName>kinect2_optical_frame1</frameName>
+            <pointCloudCutoff>0.5</pointCloudCutoff>
+            <pointCloudCutoffMax>2.0</pointCloudCutoffMax>
+        </plugin>
+        <always_on>true</always_on>
+        <update_rate>1.0</update_rate>
+    </sensor>
+</gazebo>
 </robot>

File: traxxas_description/urdf/robot05.urdf.xacro (robot description, xacro)
@@ -83,5 +83,5 @@
     <color rgba="0 1 0 1"/>
   </material>
-  <xacro:include filename="$(find traxxas_description)/urdf/robot04.gazebo.macro.xacro"/>
+  <xacro:include filename="$(find traxxas_description)/urdf/robot05.gazebo.macro.xacro"/>
   <!-- Null inertial element. This is needed to make the model work with
        Gazebo. -->
@@ -345,68 +345,56 @@
     </visual>
   </link>
-  <!--lane camara center -->
-  <joint name="camera_joint" type="fixed">
-    <origin xyz="0.073 0.0 0.084" rpy="0 0.6 0"/>
-    <parent link="base_link"/>
-    <child link="camera_link"/>
-  </joint>
-  <link name="camera_link">
-    <visual>
-      <geometry>
-        <box size="0.015 0.030 0.027"/>
-      </geometry>
-      <material name="camera_mat"/>
+  <!--lane kinect camara center -->
+  <joint name="kinect_joint" type="fixed">
+    <origin xyz="0.073 0.0 0.12" rpy="0.6 0.0 1.5708"/>
+    <parent link="base_link"/>
+    <child link="kinect_link"/>
+  </joint>
+  <link name="kinect_link">
+    <origin xyz="0 0 0" rpy="0 0 0"/>
+    <visual>
+      <origin xyz="0 0 0" rpy="0 0 0"/>
+      <geometry>
+        <mesh filename="package://traxxas_description/meshes/kinect.dae"/>
+      </geometry>
     </visual>
     <collision>
-      <origin xyz="0.005 0.0 0.013" rpy="0 0 0"/>
-      <geometry>
-        <box size="0.015 0.030 0.027"/>
+      <geometry>
+        <box size="0.06 0.30 0.07"/>
       </geometry>
     </collision>
   </link>
-  <joint name="camera_rgb_joint" type="fixed">
-    <origin xyz="0.003 0.0 0.45" rpy="0 0 0"/>
-      <parent link="camera_link"/>
-    <child link="camera_rgb_frame"/>
-  </joint>
-  <link name="camera_rgb_frame"/>
-  <joint name="camera_rgb_optical_joint" type="fixed">
-    <origin xyz="0 0 0" rpy="-1.57 0 -1.57"/>
-    <parent link="camera_rgb_frame"/>
-    <child link="camera_rgb_optical_frame"/>
-  </joint>
-  <link name="camera_rgb_optical_frame"/>
-  <!--signal camara -->
-  <joint name="camera2_joint" type="fixed">
-    <origin xyz="0.073 0.0 0.14" rpy="0 0 0"/>
-    <parent link="base_link"/>
-    <child link="camera2_link"/>
-  </joint>
-  <link name="camera2_link">
-    <visual>
-      <geometry>
-        <box size="0.015 0.030 0.027"/>
-      </geometry>
-      <material name="camera_mat"/>
+  <joint name="kinect_optical_joint" type="fixed">
+    <origin xyz="0 0 0" rpy="0 0 -1.5708"/>
+    <parent link="kinect_link"/>
+    <child link="kinect_optical_frame"/>
+  </joint>
+  <link name="kinect_optical_frame"/>
+  <!--signal kinect camara -->
+  <joint name="kinect2_joint" type="fixed">
+    <origin xyz="0.073 0.0 0.24" rpy="0 0 1.5708"/>
+    <parent link="base_link"/>
+    <child link="kinect2_link"/>
+  </joint>
+  <link name="kinect2_link">
+    <origin xyz="0 0 0" rpy="0 0 0"/>
+    <visual>
+      <origin xyz="0 0 0" rpy="0 0 0"/>
+      <geometry>
+        <mesh filename="package://traxxas_description/meshes/kinect.dae"/>
+      </geometry>
     </visual>
     <collision>
-      <origin xyz="0.005 0.0 0.013" rpy="0 0 0"/>
-      <geometry>
-        <box size="0.015 0.030 0.027"/>
+      <geometry>
+        <box size="0.06 0.30 0.07"/>
       </geometry>
     </collision>
   </link>
-  <joint name="camera2_rgb_joint" type="fixed">
-    <origin xyz="0.003 0.0 0.45" rpy="0 0 0"/>
-    <parent link="camera2_link"/>
-    <child link="camera2_rgb_frame"/>
-  </joint>
-  <link name="camera2_rgb_frame"/>
-  <joint name="camera2_rgb_optical_joint" type="fixed">
-    <origin xyz="0 0 0" rpy="-1.57 0 -1.57"/>
-    <parent link="camera2_rgb_frame"/>
-    <child link="camera2_rgb_optical_frame"/>
-  </joint>
-  <link name="camera2_rgb_optical_frame"/>
+  <joint name="kinect2_optical_joint" type="fixed">
+    <origin xyz="0 0 0" rpy="0 0 -1.5708"/>
+    <parent link="kinect2_link"/>
+    <child link="kinect2_optical_frame"/>
+  </joint>
+  <link name="kinect2_optical_frame" />
   <!--lane camara left -->
   <joint name="cameral_joint" type="fixed">
