Commit message: #32 Changed every simulation to robot 05

File: traxxas_description/urdf/robot05.urdf.xacro (robot description, xacro)
@@ -347,5 +347,5 @@
   <!--lane kinect camara center -->
   <joint name="kinect_joint" type="fixed">
-    <origin xyz="0.073 0.0 0.12" rpy="0.6 0.0 1.5708"/>
+    <origin xyz="0.07 0.0 0.38" rpy="0.1745 0.0 1.5708"/>
     <parent link="base_link"/>
     <child link="kinect_link"/>
@@ -373,5 +373,5 @@
   <!--signal kinect camara -->
   <joint name="kinect2_joint" type="fixed">
-    <origin xyz="0.073 0.0 0.24" rpy="0 0 1.5708"/>
+    <origin xyz="0.09 0.0 0.035" rpy="-0.7854 0 1.5708"/>
     <parent link="base_link"/>
     <child link="kinect2_link"/>

Commit message: I change the urdf parameters

File: traxxas_description/urdf/robot05.urdf.xacro (robot description, xacro)
@@ -347,5 +347,5 @@
   <!--lane kinect camara center -->
   <joint name="kinect_joint" type="fixed">
-    <origin xyz="0.07 0.0 0.38" rpy="0.1745 0.0 1.5708"/>
+    <origin xyz="0.07 0.0 0.38" rpy="0.38 0.0 1.5708"/>
     <parent link="base_link"/>
     <child link="kinect_link"/>
