Commit message: #120 first development in this issue, now code writs urdf to yaml files after writing

File: traxxas_description/urdf/robot05_040_038.gazebo.macro.xacro (robot description, xacro)
@@ -178,5 +178,5 @@
                 <width>1280</width>
                 <height>1024</height>
-                <format>L_INT8</format>
+                <format>R8G8B8</format>
             </image>
             <clip>
@@ -207,5 +207,5 @@
         </plugin>
         <always_on>true</always_on>
-        <update_rate>1.0</update_rate>
+        <update_rate>30.0</update_rate>
     </sensor>
 </gazebo>
@@ -219,5 +219,5 @@
                 <width>1280</width>
                 <height>1024</height>
-                <format>L_INT8</format>
+                <format>R8G8B8</format>
             </image>
             <clip>

File: traxxas_description/urdf/robot05_040_038.urdf.xacro (robot description, xacro)
@@ -83,5 +83,5 @@
     <color rgba="0 1 0 1"/>
   </material>
-  <xacro:include filename="$(find traxxas_description)/urdf/robot05.gazebo.macro.xacro"/>
+  <xacro:include filename="$(find traxxas_description)/urdf/robot05_040_038.gazebo.macro.xacro"/>
   <!-- Null inertial element. This is needed to make the model work with
        Gazebo. -->
@@ -347,5 +347,5 @@
   <!--lane kinect camara center -->
   <joint name="kinect_joint" type="fixed">
-    <origin xyz="0.073 0.0 0.12" rpy="0.5 0.0 1.5708"/>
+    <origin xyz="0.07 0.0 0.38" rpy="0.40 0.0 1.5708"/>
     <parent link="base_link"/>
     <child link="kinect_link"/>
@@ -373,5 +373,5 @@
   <!--signal kinect camara -->
   <joint name="kinect2_joint" type="fixed">
-    <origin xyz="0.073 0.0 0.24" rpy="0 0 1.5708"/>
+    <origin xyz="0.09 0.0 0.035" rpy="-0.7854 0 1.5708"/>
     <parent link="base_link"/>
     <child link="kinect2_link"/>
