Commit message: #143 Simulation totally implemented, general bringup created, sensor and arduino bringup started

File: prometheus_description/urdf/prometheus_ackermann.urdf.xacro (robot description, xacro)
@@ -15,4 +15,5 @@
     <xacro:property name="height_offset" value="0"/>
     <xacro:property name="wheel_radius" value="0.06" /> <!-- Link 1 -->
+    <xacro:property name="board_height" value="0.15" /> <!-- Link 1 -->
     <xacro:property name="thickness" value="0.032" /> <!-- Link 2 -->
     <!--  we need two because the car isn't a square-->
@@ -21,10 +22,10 @@
     <xacro:property name="steer_offset" value="0.02" /> <!-- Link 1 -->
     <!-- Add car macro -->
-    <xacro:prometheus length="${length}" width="${width}" height="${height}" wheel_radius="${wheel_radius}"/>
+    <xacro:prometheus length="${length}" width="${width}" height="${height}" board_height="${board_height}" wheel_radius="${wheel_radius}"/>
     <!-- Add sensors-->
-    <xacro:kinect name="top_front_camera" x="0.3" y="0" z="0.6" roll="0" pitch="0.4" yaw="0"/>
+    <xacro:kinect name="top_front_camera" x= "-0.22" y="0" z="0.6" roll="0" pitch="0.4" yaw="0"/>
     <xacro:kinect name="bottom_front_camera" x="0.3" y="0" z="0.2" roll="0" pitch="0" yaw="0"/>
-    <xacro:usb_cam name="top_left_camera" x="0.3" y="0.1" z="0.8" roll="0" pitch="0" yaw="0"/>
-    <xacro:usb_cam name="top_right_camera" x="0.3" y="-0.1" z="0.8" roll="0" pitch="0" yaw="-1.5708"/>
+    <xacro:usb_cam name="top_left_camera" x="-0.28" y="0.025" z="0.7" roll="0" pitch="-0.3" yaw="0"/>
+    <xacro:usb_cam name="top_right_camera" x="-0.28" y="-0.025" z="0.7" roll="0" pitch="-0.3" yaw="-1.5708"/>
     <!-- Add gazebo functionalities-->
     <xacro:include filename="$(find prometheus_description)/urdf/prometheus.gazebo.macro.xacro"/>

File: prometheus_description/urdf/prometheus_ackermann_macro.urdf.xacro (robot description, xacro)
@@ -5,5 +5,5 @@
     <xacro:include filename="$(find pointgrey_camera_description)/urdf/pointgrey_flea3.urdf.xacro"/>
     <xacro:include filename="$(find lms1xx)/urdf/sick_lms1xx.urdf.xacro"/>
-    <xacro:macro name="prometheus" params="length width wheel_radius height">
+    <xacro:macro name="prometheus" params="length width wheel_radius board_height height">
         <!-- Links: inertial,visual,collision -->
         <link name="base_link">
@@ -18,5 +18,5 @@
             <visual>
                 <!-- <origin xyz="${length/2} ${-width/2-0.15} ${-wheel_radius+0.05}" rpy="0 0 0"/> -->
-                <origin xyz="${length/2} ${-width+0.09} ${wheel_radius}" rpy="${90 * deg_to_rad} 0 ${180 * deg_to_rad}"/>
+                <origin xyz="${length/2} ${-width/2} ${board_height}" rpy="${90 * deg_to_rad} 0 ${180 * deg_to_rad}"/>
                 <geometry>
                     <mesh filename="file:///$(find prometheus_description)/meshes/chassis.dae"/>
@@ -40,34 +40,8 @@
         </link>
         <joint name="base_footprint_joint" type="fixed">
-            <origin xyz="0 0 ${wheel_radius}" rpy="0 0 0"/>
+            <origin xyz="0 0 0" rpy="0 0 0"/>
             <child link="base_link"/>
             <parent link="base_footprint"/>
         </joint>
     </xacro:macro>
-    <xacro:macro name="kinect" params="name x y z roll pitch yaw">
-        <joint name="kinect_${name}_joint" type="fixed">
-            <origin xyz="${x} ${y} ${z}" rpy="${roll} ${pitch} ${yaw}"/>
-            <parent link="base_link"/>
-            <child link="kinect_${name}_link"/>
-        </joint>
-        <link name="kinect_${name}_link">
-            <origin xyz="0 0 0" rpy="0 0 0"/>
-            <visual>
-                <origin xyz="0 0 0" rpy="0 0 0"/>
-                <geometry>
-                    <mesh filename="package://traxxas_description/meshes/kinect.dae"/>
-                </geometry>
-            </visual>
-            <collision>
-                <geometry>
-                    <box size="0.06 0.30 0.07"/>
-                </geometry>
-            </collision>
-        </link>
-        <joint name="kinect_${name}_optical_joint" type="fixed">
-            <origin xyz="0 0 0" rpy="0 0 -1.5708"/>
-            <parent link="kinect_${name}_link"/>
-            <child link="kinect_${name}_optical_frame"/>
-        </joint>
-    </xacro:macro>
 </robot>
