Commit message: #143 added compatibility between real and simulated environment

File: prometheus_description/urdf/prometheus.gazebo.macro.xacro (robot description, xacro)
@@ -4,5 +4,5 @@
         <sensor name="kinect" type="depth">
             <!-- openni plugin has the x pointing towards the scene, so rotate to have z -->
-            <pose frame="world">0.0 0.0 0.0 0.0 0.0 0.0</pose>
+            <pose frame="world">0.0 0.0 0.0 -1.5708 0.0 1.5708</pose>
             <camera>
                 <horizontal_fov>0.74839718</horizontal_fov>
@@ -28,10 +28,10 @@
                 will control the frame rate. -->
                 <updateRate>0.0</updateRate>
-                <cameraName>kinect_test</cameraName>
-                <imageTopicName>/top_front_camera/image_raw</imageTopicName>
-                <cameraInfoTopicName>/top_front_camera/camera_info</cameraInfoTopicName>
-                <depthImageTopicName>/top_front_camera/image_raw_depth</depthImageTopicName>
-                <depthImageInfoTopicName>/top_front_camera/camera_info</depthImageInfoTopicName>
-                <pointCloudTopicName>/top_front_camera/3d_cloud</pointCloudTopicName>
+                <cameraName>top_front_camera</cameraName>
+                <imageTopicName>/top_front_camera/rgb/image_color</imageTopicName>
+                <cameraInfoTopicName>/top_front_camera/rgb/camera_info</cameraInfoTopicName>
+                <depthImageTopicName>/top_front_camera/depth_registered/image</depthImageTopicName>
+                <depthImageInfoTopicName>/top_front_camera/depth_registered/camera_info</depthImageInfoTopicName>
+                <pointCloudTopicName>/top_front_camera/depth_registered/points</pointCloudTopicName>
                 <frameName>top_front_camera_optical_frame</frameName>
                 <pointCloudCutoff>0.5</pointCloudCutoff>
@@ -45,5 +45,5 @@
         <sensor name="kinect" type="depth">
             <!-- openni plugin has the x pointing towards the scene, so rotate to have z -->
-            <pose frame="world">0.0 0.0 0.0 0.0 0.0 0.0</pose>
+            <pose frame="world">0.0 0.0 0.0 -1.5708 0.0 1.5708</pose>
             <camera>
                 <horizontal_fov>0.74839718</horizontal_fov>
@@ -69,10 +69,10 @@
                 will control the frame rate. -->
                 <updateRate>0.0</updateRate>
-                <cameraName>kinect_test</cameraName>
-                <imageTopicName>/bottom_front_camera/image_raw</imageTopicName>
-                <cameraInfoTopicName>/bottom_front_camera/camera_info</cameraInfoTopicName>
-                <depthImageTopicName>/bottom_front_camera/image_raw_depth</depthImageTopicName>
-                <depthImageInfoTopicName>/bottom_front_camera/camera_info</depthImageInfoTopicName>
-                <pointCloudTopicName>/bottom_front_camera/3d_cloud</pointCloudTopicName>
+                <cameraName>bottom_front_camera</cameraName>
+                <imageTopicName>/bottom_front_camera/rgb/image_color</imageTopicName>
+                <cameraInfoTopicName>/bottom_front_camera/rgb/camera_info</cameraInfoTopicName>
+                <depthImageTopicName>/bottom_front_camera/depth_registered/image</depthImageTopicName>
+                <depthImageInfoTopicName>/bottom_front_camera/depth_registered/camera_info</depthImageInfoTopicName>
+                <pointCloudTopicName>/bottom_front_camera/depth_registered/points</pointCloudTopicName>
                 <frameName>bottom_front_camera_optical_frame</frameName>
                 <pointCloudCutoff>0.5</pointCloudCutoff>
@@ -104,6 +104,6 @@
             <cameraName>top_left_camera</cameraName>
             <frameName>top_left_camera_rgb_optical_frame</frameName>
-            <imageTopicName>top_left_camera/image_raw</imageTopicName>
-            <cameraInfoTopicName>top_left_camera/camera_info</cameraInfoTopicName>
+            <imageTopicName>image_raw</imageTopicName>
+            <cameraInfoTopicName>camera_info</cameraInfoTopicName>
             <hackBaseline>0.07</hackBaseline>
             <distortionK1>0.0</distortionK1>
@@ -136,6 +136,6 @@
             <cameraName>top_right_camera</cameraName>
             <frameName>top_right_camera_rgb_optical_frame</frameName>
-            <imageTopicName>top_right_camera/image_raw</imageTopicName>
-            <cameraInfoTopicName>top_right_camera/camera_info</cameraInfoTopicName>
+            <imageTopicName>image_raw</imageTopicName>
+            <cameraInfoTopicName>camera_info</cameraInfoTopicName>
             <hackBaseline>0.07</hackBaseline>
             <distortionK1>0.0</distortionK1>

File: prometheus_description/urdf/sensors_macro.urdf.xacro (robot description, xacro)
@@ -11,5 +11,4 @@
             <visual>
                 <origin xyz="0 0 0" rpy="0 0 1.5708"/>
-                <!-- <origin xyz="0 0 0" rpy="0 0 0"/> -->
                 <geometry>
                     <mesh filename="package://prometheus_description/meshes/kinect.dae"/>

Commit message: #176 Correction of point transformation error

File: prometheus_description/urdf/prometheus.gazebo.macro.xacro (robot description, xacro)
@@ -1,5 +1,5 @@
 <?xml version="1.0"?>
 <robot name="prometheus_gazebo" xmlns:xacro="http://ros.org/wiki/xacro">
-    <gazebo reference="top_front_camera_optical_frame">
+    <gazebo reference="top_front_camera_link">
         <sensor name="kinect" type="depth">
             <!-- openni plugin has the x pointing towards the scene, so rotate to have z -->
@@ -34,5 +34,5 @@
                 <depthImageInfoTopicName>/top_front_camera/depth_registered/camera_info</depthImageInfoTopicName>
                 <pointCloudTopicName>/top_front_camera/depth_registered/points</pointCloudTopicName>
-                <frameName>top_front_camera_optical_frame</frameName>
+                <frameName>top_front_camera_link</frameName>
                 <pointCloudCutoff>0.5</pointCloudCutoff>
                 <pointCloudCutoffMax>2.0</pointCloudCutoffMax>
@@ -42,5 +42,5 @@
         </sensor>
     </gazebo>
-    <gazebo reference="bottom_front_camera_optical_frame">
+    <gazebo reference="bottom_front_camera_link">
         <sensor name="kinect" type="depth">
             <!-- openni plugin has the x pointing towards the scene, so rotate to have z -->
@@ -75,5 +75,5 @@
                 <depthImageInfoTopicName>/bottom_front_camera/depth_registered/camera_info</depthImageInfoTopicName>
                 <pointCloudTopicName>/bottom_front_camera/depth_registered/points</pointCloudTopicName>
-                <frameName>bottom_front_camera_optical_frame</frameName>
+                <frameName>bottom_front_camera_link</frameName>
                 <pointCloudCutoff>0.5</pointCloudCutoff>
                 <pointCloudCutoffMax>2.0</pointCloudCutoffMax>
@@ -83,5 +83,5 @@
         </sensor>
     </gazebo>
-    <gazebo reference="top_left_camera_rgb_optical_frame">
+    <gazebo reference="top_left_camera_link">
         <sensor type="camera" name="Usb Camera">
         <always_on>true</always_on>
@@ -103,5 +103,5 @@
             <updateRate>30.0</updateRate>
             <cameraName>top_left_camera</cameraName>
-            <frameName>top_left_camera_rgb_optical_frame</frameName>
+            <frameName>top_left_camera_link</frameName>
             <imageTopicName>image_raw</imageTopicName>
             <cameraInfoTopicName>camera_info</cameraInfoTopicName>
@@ -115,5 +115,12 @@
         </sensor>
     </gazebo>
-    <gazebo reference="top_right_camera_rgb_optical_frame">
+    Pull requests
+    Issues
+    Codespaces
+    Marketplace
+    Explore
+    @manuelgitgomes
+    Top Repositories
+        <gazebo reference="top_right_camera_link">
         <sensor type="camera" name="Usb Camera">
         <always_on>true</always_on>
@@ -135,5 +142,5 @@
             <updateRate>30.0</updateRate>
             <cameraName>top_right_camera</cameraName>
-            <frameName>top_right_camera_rgb_optical_frame</frameName>
+            <frameName>top_right_camera_link</frameName>
             <imageTopicName>image_raw</imageTopicName>
             <cameraInfoTopicName>camera_info</cameraInfoTopicName>

File: prometheus_description/urdf/sensors_macro.urdf.xacro (robot description, xacro)
@@ -22,5 +22,5 @@
         </link>
         <joint name="${name}_optical_joint" type="fixed">
-            <origin xyz="0 0 0" rpy="0 0 0"/>
+            <origin xyz="0 0 0" rpy="-1.5708 0 -1.5708"/>
             <parent link="${name}_link"/>
             <child link="${name}_optical_frame"/>
@@ -48,5 +48,5 @@
         </link>
         <joint name="${name}_rgb_optical_joint" type="fixed">
-            <origin xyz="0 0 0" rpy="0 0 0"/>
+            <origin xyz="0 0 0" rpy="-1.5708 0 -1.5708"/>
             <parent link="${name}_link"/>
             <child link="${name}_rgb_optical_frame"/>
